File: hardware/main-board/PowerCircuit.kicad_sch (KiCad schematic)
At the start: 17 parts, among them U24 LM2776, U25 TPS54202DDC

Commit message: Added TPS55285 Foot and Sym
Parts:
- added Cinx1, Cinx2: 100n, symbol Device:C
- added L1: 10u, symbol Device:L
- added U1: XTPS55285VALR, VAL0015A-MFG, symbol SeniorDesign:XTPS55285VALR
- renumbered C11 to C?, C9 to C?, C10 to C?, Cboot to Cboot?, Cff to Cff?, Cin1 to Cin?, Cin3 to Cin?, Cin2 to Cin?, Cinx to Cinx?, Cout1 to Cout?, Cout2 to Cout?, Coutx to Coutx?, L1 to L?, Rfbb to Rfbb?, Rfbt to Rfbt?, U24 to U?, U25 to U?
Connections:
- net GNDPWR: now also U1.7 (PGND)
- new net: Cinx2.1, L1.2, U1.6 (SW1)
- new net: Cinx2.2, U1.15 (BOOT1)
- new net: Cinx1.1, L1.1, U1.8 (SW2)
- new net: Cinx1.2, U1.14 (BOOT2)
- new net GNDA: U1.12 (AGND)
Other:
- note added: "Switching Buck-Boost Converter"
