File: hardware/main-board/MainBoard.kicad_sch (KiCad schematic)
At the start: 14 parts, among them J4 Conn_01x03_Pin, J5 Conn_01x03_Pin, J6 Conn_01x03_Pin, J7 Conn_01x03_Pin, SW2 SW_SP3T, SW3 SW_SP3T, U0 TL071, U1 MT8816AF1, U1 TL071, U13 TL081, U2 TL071, U3 TL071

Commit message: fortnite info cache
Parts:
- renumbered F2 to F1, F1 to F2, J4 to J1, J5 to J2, J7 to J3, J6 to J4, SW3 to SW1, U13 to U2, U0 to U3, U1 to U4, U2 to U5, U3 to U6
Changed lines of the file:
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@@
 	(rectangle
 		(start 120.65 78.74)
-		(end 175.26 196.85)
+		(end 175.26 195.58)
 		(stroke
 			(width 0)
@@
 		(on_board yes)
 		(dnp no)
-		(property "Reference" "U0"
+		(property "Reference" "U3"
 			(at 260.35 35.4898 0)
 			(effects
@@
 			(project "MainBoard"
 				(path "/5dd933ff-bc57-4741-8957-85d8c6e75130"
-					(reference "U0")
+					(reference "U3")
 					(unit 1)
 				)
@@
 		(dnp no)
 		(fields_autoplaced yes)
-		(property "Reference" "#PWR028"
+		(property "Reference" "#PWR05"
 			(at 186.69 45.72 0)
 			(effects
@@
 			(project ""
 				(path "/5dd933ff-bc57-4741-8957-85d8c6e75130"
-					(reference "#PWR028")
+					(reference "#PWR05")
 					(unit 1)
 				)
@@
 		(dnp no)
 		(fields_autoplaced yes)
-		(property "Reference" "#PWR011"
+		(property "Reference" "#PWR014"
 			(at 245.11 114.3 0)
 			(effects
@@
 			(project "MainBoard"
 				(path "/5dd933ff-bc57-4741-8957-85d8c6e75130"
-					(reference "#PWR011")
+					(reference "#PWR014")
 					(unit 1)
 				)
@@
 		(dnp no)
 		(fields_autoplaced yes)
-		(property "Reference" "#PWR02"
+		(property "Reference" "#PWR08"
 			(at 245.11 34.29 0)
 			(effects
@@
 			(project ""
 				(path "/5dd933ff-bc57-4741-8957-85d8c6e75130"
-					(reference "#PWR02")
+					(reference "#PWR08")
 					(unit 1)
 				)
@@
 		(dnp no)
 		(fields_autoplaced yes)
-		(property "Reference" "J5"
+		(property "Reference" "J2"
 			(at 50.165 104.14 0)
 			(effects
@@
 			(project "MainBoard"
 				(path "/5dd933ff-bc57-4741-8957-85d8c6e75130"
-					(reference "J5")
+					(reference "J2")
 					(unit 1)
 				)
@@
 		(dnp no)
 		(fields_autoplaced yes)
-		(property "Reference" "#PWR057"
+		(property "Reference" "#PWR06"
 			(at 212.09 110.49 0)
 			(effects
@@
 			(project ""
 				(path "/5dd933ff-bc57-4741-8957-85d8c6e75130"
-					(reference "#PWR057")
+					(reference "#PWR06")
 					(unit 1)
 				)
@@
 		(dnp no)
 		(fields_autoplaced yes)
-		(property "Reference" "#PWR08"
+		(property "Reference" "#PWR012"
 			(at 245.11 87.63 0)
 			(effects
@@
 			(project "MainBoard"
 				(path "/5dd933ff-bc57-4741-8957-85d8c6e75130"
-					(reference "#PWR08")
+					(reference "#PWR012")
 					(unit 1)
 				)
@@
 		(dnp no)
 		(fields_autoplaced yes)
-		(property "Reference" "J4"
+		(property "Reference" "J1"
 			(at 50.165 90.17 0)
 			(effects
@@
 			(project ""
 				(path "/5dd933ff-bc57-4741-8957-85d8c6e75130"
-					(reference "J4")
+					(reference "J1")
 					(unit 1)
 				)
@@
 		(on_board yes)
 		(dnp no)
-		(property "Reference" "#PWR012"
+		(property "Reference" "#PWR015"
 			(at 248.92 125.73 0)
 			(effects
@@
 			(project "MainBoard"
 				(path "/5dd933ff-bc57-4741-8957-85d8c6e75130"
-					(reference "#PWR012")
+					(reference "#PWR015")
 					(unit 1)
 				)
@@
 		(dnp no)
 		(fields_autoplaced yes)
-		(property "Reference" "#PWR027"
+		(property "Reference" "#PWR04"
 			(at 186.69 38.1 0)
 			(effects
@@
 			(project ""
 				(path "/5dd933ff-bc57-4741-8957-85d8c6e75130"
-					(reference "#PWR027")
+					(reference "#PWR04")
 					(unit 1)
 				)
@@
 		(dnp no)
 		(fields_autoplaced yes)
-		(property "Reference" "#PWR05"
+		(property "Reference" "#PWR010"
 			(at 245.11 60.96 0)
 			(effects
@@
 			(project "MainBoard"
 				(path "/5dd933ff-bc57-4741-8957-85d8c6e75130"
-					(reference "#PWR05")
+					(reference "#PWR010")
 					(unit 1)
 				)
@@
 		(dnp no)
 		(fields_autoplaced yes)
-		(property "Reference" "U1"
+		(property "Reference" "U4"
 			(at 260.35 62.1598 0)
 			(effects
@@
 			(project "MainBoard"
 				(path "/5dd933ff-bc57-4741-8957-85d8c6e75130"
-					(reference "U1")
+					(reference "U4")
 					(unit 1)
 				)
@@
 		(dnp no)
 		(fields_autoplaced yes)
-		(property "Reference" "U3"
+		(property "Reference" "U6"
 			(at 260.35 115.4998 0)
 			(effects
@@
 			(project "MainBoard"
 				(path "/5dd933ff-bc57-4741-8957-85d8c6e75130"
-					(reference "U3")
+					(reference "U6")
 					(unit 1)
 				)
@@
 		(on_board yes)
 		(dnp no)
-		(property "Reference" "#PWR03"
+		(property "Reference" "#PWR09"
 			(at 248.92 45.72 0)
 			(effects
@@
 			(project ""
 				(path "/5dd933ff-bc57-4741-8957-85d8c6e75130"
-					(reference "#PWR03")
+					(reference "#PWR09")
 					(unit 1)
 				)
@@
 		(dnp no)
 		(fields_autoplaced yes)
-		(property "Reference" "J6"
+		(property "Reference" "J4"
 			(at 80.645 173.99 0)
 			(effects
@@
 			(project "MainBoard"
 				(path "/5dd933ff-bc57-4741-8957-85d8c6e75130"
-					(reference "J6")
+					(reference "J4")
 					(unit 1)
 				)
@@
 		(on_board yes)
 		(dnp no)
-		(property "Reference" "#PWR09"
+		(property "Reference" "#PWR013"
 			(at 248.92 99.06 0)
 			(effects
@@
 			(project "MainBoard"
 				(path "/5dd933ff-bc57-4741-8957-85d8c6e75130"
-					(reference "#PWR09")
+					(reference "#PWR013")
 					(unit 1)
 				)
@@
 		(dnp no)
 		(fields_autoplaced yes)
-		(property "Reference" "SW3"
+		(property "Reference" "SW1"
 			(at 50.8 147.32 0)
 			(effects
@@
 			(project "MainBoard"
 				(path "/5dd933ff-bc57-4741-8957-85d8c6e75130"
-					(reference "SW3")
+					(reference "SW1")
 					(unit 1)
 				)
@@
 		(dnp no)
 		(fields_autoplaced yes)
-		(property "Reference" "F1"
+		(property "Reference" "F2"
 			(at 214.63 130.8099 0)
 			(effects
@@
 			(project ""
 				(path "/5dd933ff-bc57-4741-8957-85d8c6e75130"
-					(reference "F1")
+					(reference "F2")
 					(unit 1)
 				)
@@
 		(on_board yes)
 		(dnp no)
-		(property "Reference" "U2"
+		(property "Reference" "U5"
 			(at 260.35 88.138 0)
 			(effects
@@
 			(project "MainBoard"
 				(path "/5dd933ff-bc57-4741-8957-85d8c6e75130"
-					(reference "U2")
+					(reference "U5")
 					(unit 1)
 				)
@@
 		(dnp no)
 		(fields_autoplaced yes)
-		(property "Reference" "#PWR098"
+		(property "Reference" "#PWR02"
 			(at 71.12 179.07 0)
 			(effects
@@
 			(project ""
 				(path "/5dd933ff-bc57-4741-8957-85d8c6e75130"
-					(reference "#PWR098")
+					(reference "#PWR02")
 					(unit 1)
 				)
@@
 		(dnp no)
 		(fields_autoplaced yes)
-		(property "Reference" "#PWR056"
+		(property "Reference" "#PWR07"
 			(at 212.09 133.35 0)
 			(effects
@@
 			(project ""
 				(path "/5dd933ff-bc57-4741-8957-85d8c6e75130"
-					(reference "#PWR056")
+					(reference "#PWR07")
 					(unit 1)
 				)
@@
 		(dnp no)
 		(fields_autoplaced yes)
-		(property "Reference" "U13"
+		(property "Reference" "U2"
 			(at 198.12 35.4898 0)
 			(effects
@@
 			(project ""
 				(path "/5dd933ff-bc57-4741-8957-85d8c6e75130"
-					(reference "U13")
+					(reference "U2")
 					(unit 1)
 				)
@@
 		(dnp no)
 		(fields_autoplaced yes)
-		(property "Reference" "#PWR097"
+		(property "Reference" "#PWR01"
 			(at 59.69 121.92 0)
 			(effects
@@
 			(project ""
 				(path "/5dd933ff-bc57-4741-8957-85d8c6e75130"
-					(reference "#PWR097")
+					(reference "#PWR01")
 					(unit 1)
 				)
@@
 		(dnp no)
 		(fields_autoplaced yes)
-		(property "Reference" "J7"
+		(property "Reference" "J3"
 			(at 82.55 154.9399 0)
 			(effects
@@
 			(project "MainBoard"
 				(path "/5dd933ff-bc57-4741-8957-85d8c6e75130"
-					(reference "J7")
+					(reference "J3")
 					(unit 1)
 				)
@@
 		(dnp no)
 		(fields_autoplaced yes)
-		(property "Reference" "#PWR058"
+		(property "Reference" "#PWR03"
 			(at 182.88 116.84 0)
 			(effects
@@
 			(project ""
 				(path "/5dd933ff-bc57-4741-8957-85d8c6e75130"
-					(reference "#PWR058")
+					(reference "#PWR03")
 					(unit 1)
 				)
@@
 		(dnp no)
 		(fields_autoplaced yes)
-		(property "Reference" "F2"
+		(property "Reference" "F1"
 			(at 214.63 113.0299 0)
 			(effects
@@
 			(project "MainBoard"
 				(path "/5dd933ff-bc57-4741-8957-85d8c6e75130"
-					(reference "F2")
+					(reference "F1")
 					(unit 1)
 				)
@@
 		(on_board yes)
 		(dnp no)
-		(property "Reference" "#PWR06"
+		(property "Reference" "#PWR011"
 			(at 248.92 72.39 0)
 			(effects
@@
 			(project "MainBoard"
 				(path "/5dd933ff-bc57-4741-8957-85d8c6e75130"
-					(reference "#PWR06")
+					(reference "#PWR011")
 					(unit 1)
 				)
