File: hardware/main-board/standard_cell.kicad_sch (KiCad schematic)
At the start: 13 parts, among them J5 Conn_01x02_Pin, U10 TL071, U11 MT8816AF1, U12 MT8816AF1, U7 TL071, U8 AD5263BRUZ200, U9 AD5263BRUZ200

Commit message: Updated Footprints and Controls
Parts:
- C1, C2, C3, C4: footprint (none) -> Capacitor_SMD:C_0603_1608Metric_Pad1.08x0.95mm_HandSolder
- U10, U7: footprint (none) -> Package_SO:SOIC-8_3.9x4.9mm_P1.27mm
- U8, U9: footprint AD5263BRUZ200:SOP65P640X120-24N -> SeniorDesignFP:SOP65P640X120-24N
Changed lines of the file:
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@@
 			)
 		)
-		(property "Footprint" "AD5263BRUZ200:SOP65P640X120-24N"
+		(property "Footprint" "SeniorDesignFP:SOP65P640X120-24N"
 			(at 132.08 227.076 0)
 			(effects
@@
 			)
 		)
-		(property "Footprint" "AD5263BRUZ200:SOP65P640X120-24N"
+		(property "Footprint" "SeniorDesignFP:SOP65P640X120-24N"
 			(at 133.35 138.176 0)
 			(effects
@@
 			)
 		)
-		(property "Footprint" "AD5263BRUZ200:SOP65P640X120-24N"
+		(property "Footprint" "SeniorDesignFP:SOP65P640X120-24N"
 			(at 133.35 197.866 0)
 			(effects
@@
 			)
 		)
-		(property "Footprint" ""
+		(property "Footprint" "Package_SO:SOIC-8_3.9x4.9mm_P1.27mm"
 			(at 114.3 31.75 0)
 			(effects
@@
 			)
 		)
-		(property "Footprint" ""
+		(property "Footprint" "Capacitor_SMD:C_0603_1608Metric_Pad1.08x0.95mm_HandSolder"
 			(at 147.0152 72.39 0)
 			(effects
@@
 			)
 		)
-		(property "Footprint" "AD5263BRUZ200:SOP65P640X120-24N"
+		(property "Footprint" "SeniorDesignFP:SOP65P640X120-24N"
 			(at 173.99 167.386 0)
 			(effects
@@
 			)
 		)
-		(property "Footprint" "AD5263BRUZ200:SOP65P640X120-24N"
+		(property "Footprint" "SeniorDesignFP:SOP65P640X120-24N"
 			(at 173.99 138.176 0)
 			(effects
@@
 			)
 		)
-		(property "Footprint" "AD5263BRUZ200:SOP65P640X120-24N"
+		(property "Footprint" "SeniorDesignFP:SOP65P640X120-24N"
 			(at 173.99 197.866 0)
 			(effects
@@
 			)
 		)
-		(property "Footprint" ""
+		(property "Footprint" "Capacitor_SMD:C_0603_1608Metric_Pad1.08x0.95mm_HandSolder"
 			(at 166.0652 72.39 0)
 			(effects
@@
 			)
 		)
-		(property "Footprint" "AD5263BRUZ200:SOP65P640X120-24N"
+		(property "Footprint" "SeniorDesignFP:SOP65P640X120-24N"
 			(at 173.99 225.806 0)
 			(effects
@@
 			)
 		)
-		(property "Footprint" ""
+		(property "Footprint" "Capacitor_SMD:C_0603_1608Metric_Pad1.08x0.95mm_HandSolder"
 			(at 186.3852 72.39 0)
 			(effects
@@
 			)
 		)
-		(property "Footprint" "AD5263BRUZ200:SOP65P640X120-24N"
+		(property "Footprint" "SeniorDesignFP:SOP65P640X120-24N"
 			(at 132.08 168.656 0)
 			(effects
@@
 			)
 		)
-		(property "Footprint" ""
+		(property "Footprint" "Capacitor_SMD:C_0603_1608Metric_Pad1.08x0.95mm_HandSolder"
 			(at 126.6952 72.39 0)
 			(effects
@@
 			)
 		)
-		(property "Footprint" ""
+		(property "Footprint" "Package_SO:SOIC-8_3.9x4.9mm_P1.27mm"
 			(at 49.53 31.75 0)
 			(effects
