File: hardware/main-board/standard_cell.kicad_sch (KiCad schematic)
At the start: 13 parts, among them J5 Conn_01x02_Pin, U10 TL071, U11 CD22M3494MQZ, U12 CD22M3494MQZ, U7 TL071, U8 AD5263BRUZ200, U9 AD5263BRUZ200

Commit message: finalized component list, fixed DRC errors
Parts:
- U11, U12: DKPN (none) -> CD22M3494MQZ
Changed lines of the file:
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@@
+			)
+		)
+		(property "DKPN" "CD22M3494MQZ"
+			(at 162.56 146.05 0)
+			(effects
+				(font
+					(size 1.27 1.27)
+				)
+				(hide yes)
 			)
 		)
@@
 			(at 217.17 146.05 0)
 			(effects
+				(font
+					(size 1.27 1.27)
+				)
+				(hide yes)
+			)
+		)
+		(property "DKPN" "CD22M3494MQZ"
+			(at 217.17 146.05 0)
+			(effects
