File: hardware/main-board/MainBoard.kicad_pcb (KiCad board)
At the start: 4 copper layers, 143 parts, among them J1 Conn_01x03_Pin, J10 Conn_02x05_Odd_Even, J11 Conn_01x02_Pin, J12 Barrel_Jack, J2 Conn_01x03_Pin, J3 Conn_01x03_Pin, J4 Conn_01x03_Pin, J5 Conn_01x02_Pin, J6 Conn_01x02_Pin, J7 Conn_01x02_Pin, J8 Conn_01x02_Pin, J9 USB_C_Receptacle_USB2.0_14P, SW1 SW_SP3T, SW2 SW_SP3T, SW3 SW_SPST, SW4 SW_SPST, U1 MT8816AF1, U10 TL071, U11 MT8816AF1, U12 MT8816AF1, U13 TL071, U14 AD5263BRUZ200, U15 AD5263BRUZ200, U16 TL071, U17 MT8816AF1, U18 MT8816AF1, U19 TL071, U2 TL081, U20 AD5263BRUZ200, U21 AD5263BRUZ200, U22 TL071, U23 MT8816AF1, U24 MT8816AF1, U25 TL071, U26 AD5263BRUZ200, U27 AD5263BRUZ200, U28 TL071, U29 MT8816AF1, U3 TL071, U30 MT8816AF1, U31 XTPS55285VALR, U32 TPS54202DDC, U33 LM2776, U34 74HC164, U35 FT232RL, U36 74HC164, U37 STM32F091RCTx, U38 74HC164, U4 TL071, U5 TL071, U6 TL071, U7 TL071, U8 AD5263BRUZ200, U9 AD5263BRUZ200

Commit message: designed Power PCB section layout
Parts:
- removed the U1 at (207.0, 89.5)
- removed the U11 at (241.8, 136.6)
- removed the U12 at (241.8, 151.0)
- removed the U17 at (241.8, 105.9)
- removed the U18 at (241.8, 120.2)
- removed the U23 at (208.3, 105.9)
- removed the U24 at (208.3, 120.2)
- removed the U29 at (208.3, 136.6)
- added F1: 500mA, Fuse:Fuse_0603_1608Metric_Pad1.05x0.95mm_HandSolder, F.Cu at (49.0, 155.5)
- added J13: Conn_01x02_Pin, Connector_PinHeader_1.00mm:PinHeader_1x02_P1.00mm_Horizontal, F.Cu at (74.8, 45.8)
- added U1: CD22M3494MQZ, SeniorDesignFP:PLCC44_16P66X16P66_INR-M, F.Cu at (168.7, 159.7)
- added U1: CD22M3494MQZ, SeniorDesignFP:PLCC44_16P66X16P66_INR-M, F.Cu at (99.9, 94.8)
- added U11: CD22M3494MQZ, SeniorDesignFP:PLCC44_16P66X16P66_INR-M, F.Cu at (99.9, 115.8)
- added U11: CD22M3494MQZ, SeniorDesignFP:PLCC44_16P66X16P66_INR-M, F.Cu at (145.7, 159.7)
- added U12: CD22M3494MQZ, SeniorDesignFP:PLCC44_16P66X16P66_INR-M, F.Cu at (99.9, 136.7)
- added U12: CD22M3494MQZ, SeniorDesignFP:PLCC44_16P66X16P66_INR-M, F.Cu at (145.7, 180.6)
- added U17: CD22M3494MQZ, SeniorDesignFP:PLCC44_16P66X16P66_INR-M, F.Cu at (120.8, 94.8)
- added U17: CD22M3494MQZ, SeniorDesignFP:PLCC44_16P66X16P66_INR-M, F.Cu at (122.8, 159.7)
- added U18: CD22M3494MQZ, SeniorDesignFP:PLCC44_16P66X16P66_INR-M, F.Cu at (120.8, 115.8)
- added U18: CD22M3494MQZ, SeniorDesignFP:PLCC44_16P66X16P66_INR-M, F.Cu at (122.8, 180.6)
- added U23: CD22M3494MQZ, SeniorDesignFP:PLCC44_16P66X16P66_INR-M, F.Cu at (164.7, 94.8)
- added U23: CD22M3494MQZ, SeniorDesignFP:PLCC44_16P66X16P66_INR-M, F.Cu at (120.8, 136.7)
- added U24: CD22M3494MQZ, SeniorDesignFP:PLCC44_16P66X16P66_INR-M, F.Cu at (164.7, 115.8)
- added U24: CD22M3494MQZ, SeniorDesignFP:PLCC44_16P66X16P66_INR-M, F.Cu at (141.8, 94.8)
- added U29: CD22M3494MQZ, SeniorDesignFP:PLCC44_16P66X16P66_INR-M, F.Cu at (141.8, 115.8)
- added U29: CD22M3494MQZ, SeniorDesignFP:PLCC44_16P66X16P66_INR-M, F.Cu at (99.9, 159.7)
- added U48: CD22M3494MQZ, SeniorDesignFP:PLCC44_16P66X16P66_INR-M, F.Cu at (141.8, 136.7)
- F2: value Fuse -> 500mA
- F3: renamed from F1; value Fuse -> 500mA
- U30: value MT8816AF1 -> CD22M3494MQZ; footprint SeniorDesignFP:QFP80P1200X1200X120-44N -> SeniorDesignFP:PLCC44_16P66X16P66_INR-M
- moved U30 112.4 mm to (99.9, 180.6)
- moved Cin3 44.4 mm to (23.0, 154.5), turned to 90 degrees
- moved U32 43.8 mm to (28.4, 151.9)
- moved Coutx2 43.2 mm to (39.5, 159.5), turned to -90 degrees
- moved Cin4 39.7 mm to (23.0, 159.5)
- moved Rcomp1 39.5 mm to (50.0, 154.0)
- moved L1 37.9 mm to (30.6, 159.5)
- moved F3 37.8 mm to (40.5, 162.5), turned to -90 degrees
- moved U33 37.4 mm to (46.5, 161.2), turned to -90 degrees
- moved Rfbt1 35.7 mm to (37.6, 162.2), turned to -90 degrees
- moved Cin5 35.3 mm to (23.0, 164.5), turned to 90 degrees
- moved Cinx2 33.7 mm to (47.5, 148.0), turned to -90 degrees
- moved C17 32.8 mm to (46.5, 164.2), turned to 180 degrees
- moved U37 32.6 mm to (80.5, 37.0)
- moved F2 31.0 mm to (51.5, 160.0), turned to 180 degrees
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- renumbered C30 to C20, C20 to C22, C22 to C24, C24 to C25, C25 to C26, C26 to C27, C27 to C28, C28 to C29, C29 to C30, Cboot3 to Cboot1, Cboot1 to Cboot2, Cboot2 to Cboot3, Cin4 to Cin1, Cin5 to Cin2, Cin2 to Cin4, Cin1 to Cin5, Cinx2 to Cinx1, Cinx3 to Cinx2, Cinx1 to Cinx3, Coutx2 to Coutx1, Coutx1 to Coutx2, D14 to D12, D12 to D14, F3 to F4, J9 to J10, J10 to J11, J11 to J12, J12 to J9, R6 to R1, R8 to R10, R1 to R2, R2 to R3, R7 to R4, R4 to R5, R10 to R6, R3 to R7, R5 to R8
Connections:
- U30 pad 34: /MicroController/MT_CS_5 -> /MicroController/MT_CS_8
- U31 pad 12: GNDA -> GND
- U37 pad 10: unconnected-(U37-PC2-Pad10) -> /MicroController/PC2
- U37 pad 11: unconnected-(U37-PC3-Pad11) -> /MicroController/PC3

Commit message: small edits with layout discussion
Parts:
- moved U1 106.0 mm to (90.2, 88.4)
- moved U11 106.0 mm to (67.3, 88.4)
- moved U17 106.0 mm to (44.3, 88.4)
- moved U29 106.0 mm to (21.4, 88.4)
- moved U11 106.0 mm to (21.4, 44.5)
- moved U12 106.0 mm to (21.4, 65.4)
- moved U12 106.0 mm to (67.3, 109.3)
- moved U17 106.0 mm to (42.3, 23.6)
- moved U18 106.0 mm to (42.3, 44.5)
- moved U18 106.0 mm to (44.3, 109.3)
- moved U23 106.0 mm to (86.2, 23.6)
- moved U23 106.0 mm to (42.3, 65.4)
- moved U24 106.0 mm to (86.2, 44.5)
- moved U24 106.0 mm to (63.3, 23.6)
- moved U29 106.0 mm to (63.3, 44.5)
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
Commit message: Working on that PCP
Parts:
- removed the U1 at (87.8, 145.7)
- removed the U11 at (21.4, 44.5)
- removed the U12 at (67.3, 109.3)
- moved C2 193.5 mm to (66.1, 145.0), turned to -90 degrees
- moved C4 190.3 mm to (69.5, 138.3), turned to 180 degrees
- moved D1 187.3 mm to (72.6, 138.3), turned to 180 degrees
- moved J5 184.2 mm to (75.1, 138.0), turned to 90 degrees
- moved D2 180.3 mm to (79.0, 160.0), turned to 180 degrees
- moved C3 178.1 mm to (82.1, 160.0), turned to 180 degrees
- moved U9 171.5 mm to (91.2, 157.2)
- moved U8 160.5 mm to (92.6, 139.2), turned to 180 degrees
- moved C1 152.4 mm to (108.5, 160.1), turned to 180 degrees
- moved U10 141.1 mm to (112.9, 163.8), turned to -90 degrees
- moved U7 130.9 mm to (122.9, 154.8)
- moved U12 120.4 mm to (108.1, 149.0)
- moved U37 67.5 mm to (78.0, 120.0)
- moved U11 61.6 mm to (77.0, 149.1)
Connections:
- J5 pad 1: /STD/J1_in -> /STD/J1_out
- J5 pad 2: /STD/J1_out -> /STD/J1_in
- J6 pad 1: /STD1/J1_in -> /STD1/J1_out
- J6 pad 2: /STD1/J1_out -> /STD1/J1_in
- J7 pad 1: /STD2/J1_in -> /STD2/J1_out
- J7 pad 2: /STD2/J1_out -> /STD2/J1_in
- J8 pad 1: /STD3/J1_in -> /STD3/J1_out
- J8 pad 2: /STD3/J1_out -> /STD3/J1_in
- U11 pad 28: /STD/C2_out -> /STD/R6_out
- U11 pad 29: /STD/C2_in -> /STD/R6_in
- U11 pad 30: /STD/C1_out -> /STD/R5_out
- U11 pad 31: /STD/C1_in -> /STD/R5_in
- U11 pad 8: /STD/R6_in -> /STD/C2_in
- U11 pad 9: /STD/R6_out -> /STD/C2_out
- U15 pad 22: /STD1/R6_out -> unconnected-(U15C-W2-Pad22)
- U15 pad 23: /STD1/R6_out -> unconnected-(U15C-A2-Pad23)
- U15 pad 24: /STD1/R6_in -> unconnected-(U15C-B2-Pad24)
- U15 pad 4: unconnected-(U15D-B3-Pad4) -> /STD1/R6_in
- U15 pad 5: unconnected-(U15D-A3-Pad5) -> /STD1/R6_out
- U15 pad 6: unconnected-(U15D-W3-Pad6) -> /STD1/R6_out
- U17 pad 28: /STD1/C2_out -> /STD1/R6_out
- U17 pad 29: /STD1/C2_in -> /STD1/R6_in
- U17 pad 30: /STD1/C1_out -> /STD1/R5_out
- U17 pad 31: /STD1/C1_in -> /STD1/R5_in
- U17 pad 8: /STD1/R6_in -> /STD1/C2_in
- U17 pad 9: /STD1/R6_out -> /STD1/C2_out
- U18 pad 2: /STD1/R2_in -> /STD1/R3_in
- U18 pad 24: /STD1/R1_out -> /STD1/C1_out
- U18 pad 25: /STD1/R1_in -> /STD1/C1_in
- U18 pad 26: /STD1/Op2_neg -> /STD1/Op2_pos
- U18 pad 27: /STD1/Op2_pos -> /STD1/Op2_neg
- U18 pad 29: /STD1/Op1_neg -> /STD1/Op1_pos
- U18 pad 3: /STD1/R2_out -> /STD1/R3_out
- U18 pad 30: /STD1/Op1_pos -> /STD1/Op1_neg
- U18 pad 4: /STD1/R3_in -> /STD1/R1_in
- U18 pad 5: /STD1/R3_out -> /STD1/R1_out
- U18 pad 6: /STD1/R4_in -> /STD1/R2_in
- U18 pad 7: /STD1/R4_out -> /STD1/R2_out
- U18 pad 8: /STD1/R5_in -> /STD1/R4_in
- U18 pad 9: /STD1/R5_out -> /STD1/R4_out
- U21 pad 22: /STD2/R6_out -> unconnected-(U21C-W2-Pad22)
- U21 pad 23: /STD2/R6_out -> unconnected-(U21C-A2-Pad23)
- U21 pad 24: /STD2/R6_in -> unconnected-(U21C-B2-Pad24)
- U21 pad 4: unconnected-(U21D-B3-Pad4) -> /STD2/R6_in
- U21 pad 5: unconnected-(U21D-A3-Pad5) -> /STD2/R6_out
- U21 pad 6: unconnected-(U21D-W3-Pad6) -> /STD2/R6_out
- U23 pad 28: /STD2/C2_out -> /STD2/R6_out
- U23 pad 29: /STD2/C2_in -> /STD2/R6_in
- U23 pad 30: /STD2/C1_out -> /STD2/R5_out
- U23 pad 31: /STD2/C1_in -> /STD2/R5_in
- U23 pad 8: /STD2/R6_in -> /STD2/C2_in
- U23 pad 9: /STD2/R6_out -> /STD2/C2_out
- U24 pad 2: /STD2/R2_in -> /STD2/R3_in
- U24 pad 24: /STD2/R1_out -> /STD2/C1_out
- U24 pad 25: /STD2/R1_in -> /STD2/C1_in
- U24 pad 26: /STD2/Op2_neg -> /STD2/Op2_pos
- U24 pad 27: /STD2/Op2_pos -> /STD2/Op2_neg
- U24 pad 29: /STD2/Op1_neg -> /STD2/Op1_pos
- U24 pad 3: /STD2/R2_out -> /STD2/R3_out
- U24 pad 30: /STD2/Op1_pos -> /STD2/Op1_neg
- U24 pad 4: /STD2/R3_in -> /STD2/R1_in
- U24 pad 5: /STD2/R3_out -> /STD2/R1_out
- U24 pad 6: /STD2/R4_in -> /STD2/R2_in
- U24 pad 7: /STD2/R4_out -> /STD2/R2_out
- U24 pad 8: /STD2/R5_in -> /STD2/R4_in
- U24 pad 9: /STD2/R5_out -> /STD2/R4_out
- U27 pad 22: /STD3/R6_out -> unconnected-(U27C-W2-Pad22)
- U27 pad 23: /STD3/R6_out -> unconnected-(U27C-A2-Pad23)
- U27 pad 24: /STD3/R6_in -> unconnected-(U27C-B2-Pad24)
- U27 pad 4: unconnected-(U27D-B3-Pad4) -> /STD3/R6_in
- U27 pad 5: unconnected-(U27D-A3-Pad5) -> /STD3/R6_out
- U27 pad 6: unconnected-(U27D-W3-Pad6) -> /STD3/R6_out
- U29 pad 28: /STD3/C2_out -> /STD3/R6_out
- U29 pad 29: /STD3/C2_in -> /STD3/R6_in
- U29 pad 30: /STD3/C1_out -> /STD3/R5_out
- U29 pad 31: /STD3/C1_in -> /STD3/R5_in
- U29 pad 8: /STD3/R6_in -> /STD3/C2_in
- U29 pad 9: /STD3/R6_out -> /STD3/C2_out
- U30 pad 2: /STD3/R2_in -> /STD3/R3_in
- U30 pad 24: /STD3/R1_out -> /STD3/C1_out
- U30 pad 25: /STD3/R1_in -> /STD3/C1_in
- U30 pad 26: /STD3/Op2_neg -> /STD3/Op2_pos
- U30 pad 27: /STD3/Op2_pos -> /STD3/Op2_neg
- U30 pad 29: /STD3/Op1_neg -> /STD3/Op1_pos
- U30 pad 3: /STD3/R2_out -> /STD3/R3_out
- U30 pad 30: /STD3/Op1_pos -> /STD3/Op1_neg
- U30 pad 4: /STD3/R3_in -> /STD3/R1_in
- U30 pad 5: /STD3/R3_out -> /STD3/R1_out
- U30 pad 6: /STD3/R4_in -> /STD3/R2_in
- U30 pad 7: /STD3/R4_out -> /STD3/R2_out
- U30 pad 8: /STD3/R5_in -> /STD3/R4_in
- U30 pad 9: /STD3/R5_out -> /STD3/R4_out
- U9 pad 22: /STD/R6_out -> unconnected-(U9C-W2-Pad22)
- U9 pad 23: /STD/R6_out -> unconnected-(U9C-A2-Pad23)
- U9 pad 24: /STD/R6_in -> unconnected-(U9C-B2-Pad24)
- U9 pad 4: unconnected-(U9D-B3-Pad4) -> /STD/R6_in
- U9 pad 5: unconnected-(U9D-A3-Pad5) -> /STD/R6_out
- U9 pad 6: unconnected-(U9D-W3-Pad6) -> /STD/R6_out
Routing:
- net /STD/R6_out: track 0.00 -> 6.29 mm
- net /STD/C4_out: track 0.00 -> 4.53 mm
- net /STD/R5_out: track 0.00 -> 3.66 mm
- net /STD/R5_in: track 0.00 -> 3.28 mm
- net /STD/J1_out: track 0.00 -> 3.08 mm
- net /STD/R6_in: track 0.00 -> 3.04 mm
- net /STD/J1_in: track 0.00 -> 2.97 mm
- net /STD/C3_in: track 0.00 -> 2.88 mm
- net /STD/C2_out: track 0.00 -> 2.83 mm
- net /STD/C3_out: track 0.00 -> 2.70 mm
- net /STD/C4_in: track 0.00 -> 2.65 mm
- net /STD/C2_in: track 0.00 -> 2.64 mm
- net /STD/D2_cathode: track 0.00 -> 2.57 mm
- net /STD/D1_anode: track 0.00 -> 2.55 mm
- net /STD/D1_cathode: track 0.00 -> 2.54 mm
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
Commit message: The PCB is coming together
Parts:
- removed the U17 at (42.3, 23.6)
- removed the U18 at (42.3, 44.5)
- removed the U18 at (44.3, 109.3)
- removed the U23 at (86.2, 23.6)
- removed the U23 at (42.3, 65.4)
- removed the U24 at (86.2, 44.5)
- removed the U24 at (63.3, 23.6)
- removed the U29 at (63.3, 44.5)
- removed U48: CD22M3494MQZ, SeniorDesignFP:PLCC44_16P66X16P66_INR-M
- added U18: CD22M3494MQZ, SeniorDesignFP:PLCC44_16P66X16P66_INR-M, F.Cu at (86.6, 116.2)
- added U23: CD22M3494MQZ, SeniorDesignFP:PLCC44_16P66X16P66_INR-M, F.Cu at (117.1, 78.8)
- added U24: CD22M3494MQZ, SeniorDesignFP:PLCC44_16P66X16P66_INR-M, F.Cu at (86.5, 78.8)
- C21, C22, C23, C24, C25, C26, C27, C28, C29, C30, D11, F4, FB1, R2, R3: moved to B.Cu
- J12, J13, J5, J6, J7, J8: footprint Connector_PinHeader_1.00mm:PinHeader_1x02_P1.00mm_Horizontal -> Connector_PinSocket_2.54mm:PinSocket_1x02_P2.54mm_Vertical
- moved C29 200.9 mm to (17.7, 122.0), turned to 180 degrees
- moved C30 193.7 mm to (18.5, 109.8), turned to 90 degrees
- moved SW3 193.3 mm to (22.5, 119.1)
- moved FB1 193.0 mm to (18.5, 115.5), turned to 90 degrees
- moved C28 188.4 mm to (17.7, 119.5), turned to 180 degrees
- moved C21 187.1 mm to (21.4, 109.8), turned to 90 degrees
- moved C5 184.1 mm to (75.7, 117.8), turned to 90 degrees
- moved R7 184.0 mm to (25.7, 117.1), turned to -90 degrees
- moved C23 182.7 mm to (23.9, 109.8), turned to 90 degrees
- moved U38 182.7 mm to (52.3, 111.8), turned to 180 degrees
- moved R6 182.5 mm to (38.3, 128.4), turned to -90 degrees
- moved R5 181.4 mm to (36.8, 108.1)
- moved J12 179.6 mm to (28.7, 116.1), turned to 180 degrees
- moved C13 179.6 mm to (75.4, 42.1), turned to 90 degrees
- moved U16 179.5 mm to (73.9, 125.0), turned to -90 degrees
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Connections:
- net /STD1/Input_1 renamed /STD1/Y0
- net /STD1/Input_2 renamed /STD1/Y1
- net /STD1/Input_3 renamed /STD1/Y2
- U1 pad 25: /STD2/Input_3 -> /STD2/Y2
- U1 pad 29: /STD/Input_3 -> /STD/Y2
- U1 pad 30: /STD/Input_2 -> /STD/Y1
- U1 pad 31: /STD/Input_1 -> /STD/Y0
- U1 pad 5: /STD3/Input_1 -> /STD3/Y0
- U1 pad 6: /STD3/Input_2 -> /STD3/Y1
- U1 pad 7: /STD3/Input_3 -> /STD3/Y2
- U1 pad 8: /STD2/Input_1 -> /STD2/Y0
- U1 pad 9: /STD2/Input_2 -> /STD2/Y1
- U11 pad 10: Net-(U11A-Y7) -> /STD/Y7
- U11 pad 13: Net-(U11A-Y6) -> /STD/Y6
- U11 pad 15: GND -> /STD/Y5
- U11 pad 17: Net-(U11A-Y4) -> /STD/Y4
- U11 pad 2: /STD/J1_in -> /STD/C2_in
- U11 pad 26: /STD/C3_out -> /STD/J1_out
- U11 pad 27: /STD/C3_in -> /STD/J1_in
- U11 pad 3: /STD/J1_out -> /STD/C2_out
- U11 pad 32: /STD/Input_1 -> /STD/Y0
- U11 pad 35: /STD/Input_2 -> /STD/Y1
- U11 pad 37: /STD/Input_3 -> /STD/Y2
- U11 pad 8: /STD/C2_in -> /STD/C3_in
- U11 pad 9: /STD/C2_out -> /STD/C3_out
- U12 pad 10: (no net) -> /Cell_0_Out
- U12 pad 13: (no net) -> /STD/Y2
- U12 pad 15: (no net) -> /STD/Y1
- U12 pad 17: (no net) -> /STD/Y0
- U12 pad 2: (no net) -> /STD/R3_out
- U12 pad 24: (no net) -> /STD/C1_out
- U12 pad 25: (no net) -> /STD/C1_in
- U12 pad 26: (no net) -> /STD/Op2_pos
- U12 pad 27: (no net) -> /STD/Op2_neg
- U12 pad 28: (no net) -> /STD/Op2_out
- U12 pad 29: (no net) -> /STD/Op1_neg
- U12 pad 3: (no net) -> /STD/R3_in
- U12 pad 30: (no net) -> /STD/Op1_pos
- U12 pad 31: (no net) -> /STD/Op1_out
- U12 pad 32: (no net) -> /STD/Y4
- U12 pad 34: /MicroController/MT_CS_8 -> /MicroController/MT_CS_6
- U12 pad 35: (no net) -> /STD/Y5
- U12 pad 37: (no net) -> /STD/Y6
- U12 pad 39: (no net) -> /STD/Y7
- U12 pad 4: (no net) -> /STD/R1_out
- U12 pad 5: (no net) -> /STD/R1_in
- U12 pad 6: (no net) -> /STD/R2_in
- U12 pad 7: (no net) -> /STD/R2_out
- U12 pad 8: (no net) -> /STD/R4_in
- U12 pad 9: (no net) -> /STD/R4_out
- U17 pad 10: Net-(U17A-Y7) -> /STD1/Y7
- U17 pad 13: Net-(U17A-Y6) -> /STD1/Y6
- U17 pad 15: GND -> /STD1/Y5
- U17 pad 17: Net-(U17A-Y4) -> /STD1/Y4
- U17 pad 2: /STD1/J1_in -> /STD1/C2_in
- U17 pad 26: /STD1/C3_out -> /STD1/J1_out
- U17 pad 27: /STD1/C3_in -> /STD1/J1_in
- U17 pad 3: /STD1/J1_out -> /STD1/C2_out
- U17 pad 8: /STD1/C2_in -> /STD1/C3_in
- U17 pad 9: /STD1/C2_out -> /STD1/C3_out
- U29 pad 10: Net-(U29A-Y7) -> /STD3/Y7
- U29 pad 13: Net-(U29A-Y6) -> /STD3/Y6
- U29 pad 15: GND -> /STD3/Y5
- U29 pad 17: Net-(U29A-Y4) -> /STD3/Y4
- U29 pad 2: /STD3/J1_in -> /STD3/C2_in
- U29 pad 26: /STD3/C3_out -> /STD3/J1_out
- U29 pad 27: /STD3/C3_in -> /STD3/J1_in
- U29 pad 3: /STD3/J1_out -> /STD3/C2_out
- U29 pad 32: /STD3/Input_1 -> /STD3/Y0
- U29 pad 35: /STD3/Input_2 -> /STD3/Y1
- U29 pad 37: /STD3/Input_3 -> /STD3/Y2
- U29 pad 8: /STD3/C2_in -> /STD3/C3_in
- U29 pad 9: /STD3/C2_out -> /STD3/C3_out
- U30 pad 10: Net-(U29A-Y7) -> /Cell_3_Out
- U30 pad 13: Net-(U29A-Y6) -> /STD3/Y2
- U30 pad 15: GND -> /STD3/Y1
- U30 pad 17: Net-(U29A-Y4) -> /STD3/Y0
- U30 pad 2: /STD3/R3_in -> /STD3/R3_out
- U30 pad 29: /STD3/Op1_pos -> /STD3/Op1_neg
- U30 pad 3: /STD3/R3_out -> /STD3/R3_in
- U30 pad 30: /STD3/Op1_neg -> /STD3/Op1_pos
- U30 pad 32: /STD3/Input_1 -> /STD3/Y4
- U30 pad 35: /STD3/Input_2 -> /STD3/Y5
- U30 pad 37: /STD3/Input_3 -> /STD3/Y6
- U30 pad 39: /Cell_3_Out -> /STD3/Y7
- U30 pad 4: /STD3/R1_in -> /STD3/R1_out
- U30 pad 5: /STD3/R1_out -> /STD3/R1_in
Routing:
- net GND: track 0.00 -> 105.7 mm, vias 0 -> 14
- net +3.3V: track 0.00 -> 59.5 mm, vias 0 -> 5
- net /STD/Y0: track 0.00 -> 48.3 mm, vias 0 -> 2
- net /STD3/Y0: track 0.00 -> 47.8 mm, vias 0 -> 2
- net /STD3/Y4: track 0.00 -> 46.6 mm, vias 0 -> 2
- net /STD/Y4: track 0.00 -> 46.6 mm, vias 0 -> 2
- net /STD2/Y0: track 0.00 -> 46.5 mm, vias 0 -> 2
- net /STD1/Y0: track 0.00 -> 46.2 mm, vias 0 -> 2
- net /STD2/Y4: track 0.00 -> 45.9 mm, vias 0 -> 2
- net /STD1/Y4: track 0.00 -> 45.6 mm, vias 0 -> 2
- net /STD/Y1: track 0.00 -> 41.3 mm, vias 0 -> 2
- net /STD3/Y1: track 0.00 -> 41.1 mm, vias 0 -> 2
- net /STD/Y5: track 0.00 -> 40.8 mm, vias 0 -> 2
- net /STD3/Y5: track 0.00 -> 40.7 mm, vias 0 -> 2
- net /STD2/Y5: track 0.00 -> 40.1 mm, vias 0 -> 2
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Other:
- board text added: "${REFERENCE}"

Commit message: Added wiring to cells and compacted input
Parts:
- J1, J2, J3, J4: footprint Connector_PinHeader_1.00mm:PinHeader_1x03_P1.00mm_Horizontal -> Connector_PinHeader_2.54mm:PinHeader_1x03_P2.54mm_Vertical
- J11: footprint Connector_PinHeader_1.00mm:PinHeader_2x05_P1.00mm_Horizontal -> Connector_PinHeader_2.54mm:PinHeader_2x05_P2.54mm_Vertical
- moved SW2 228.3 mm to (26.1, 78.1), turned to 180 degrees
- moved J2 209.0 mm to (16.7, 84.7)
- moved J1 202.6 mm to (16.7, 75.8)
- moved J11 201.2 mm to (26.3, 104.4), turned to -90 degrees
- moved R8 169.6 mm to (29.1, 66.9), turned to 180 degrees
- moved R1 155.8 mm to (25.9, 48.8), turned to -90 degrees
- moved R4 153.8 mm to (28.2, 48.8), turned to -90 degrees
- moved J10 153.2 mm to (16.4, 59.8), turned to -90 degrees
- moved F4 152.1 mm to (24.1, 53.7), turned to 90 degrees
- moved D9 151.3 mm to (25.9, 52.9), turned to 90 degrees
- moved D11 150.0 mm to (26.5, 53.6), turned to 90 degrees
- moved D10 149.2 mm to (28.2, 53.0), turned to 90 degrees
- moved C24 148.0 mm to (29.1, 53.3), turned to 90 degrees
- moved C20 147.0 mm to (30.4, 53.2), turned to 90 degrees
- moved R2 147.0 mm to (24.1, 58.5), turned to 0 degrees
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Routing:
- net /MicroController/MT_AX1: track 0.00 -> 314.7 mm, vias 0 -> 10
- net /MicroController/MT_AX2: track 0.00 -> 295.2 mm, vias 0 -> 12
- net /MicroController/MT_AY0: track 0.00 -> 278.7 mm, vias 0 -> 11
- net /MicroController/MT_AY1: track 0.00 -> 277.5 mm, vias 0 -> 10
- net /MicroController/MT_AY2: track 0.00 -> 148.0 mm, vias 0 -> 10
- net /MicroController/MT_AX0: track 0.00 -> 131.1 mm, vias 0 -> 2
- net /MicroController/MT_AX3: track 0.00 -> 130.1 mm, vias 0 -> 10
- net /MicroController/MT_RST: track 0.00 -> 77.9 mm, vias 0 -> 10
- net /STD3/Y2: track 35.6 -> 101.0 mm
- net /STD3/Y1: track 41.1 -> 100.5 mm
- net /MicroController/MT_DAT: track 0.00 -> 58.7 mm, vias 0 -> 4
- net /STD3/Y0: track 47.8 -> 103.1 mm
- net /Power Supply/WallAdpt: track 0.00 -> 43.4 mm
- net Net-(U35-RXD): track 23.0 -> 59.8 mm, vias 0 -> 2
- net Net-(U35-TXD): track 23.9 -> 57.1 mm, vias 0 -> 2
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