File: hardware/crossbar-fixer/crossbar-fixer.kicad_sch (KiCad schematic)
At the start: 2 parts

Commit message: I ate the fillet 'o fish
Parts:
- renumbered Fucked1 to U2
Changed lines of the file:
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@@
 		(on_board yes)
 		(dnp no)
-		(property "Reference" "Fucked1"
+		(property "Reference" "U2"
 			(at 156.21 76.2 0)
 			(effects
@@
 			(project ""
 				(path "/42dafeb3-7ab4-4fdc-a747-7ffb34623964"
-					(reference "Fucked1")
+					(reference "U2")
 					(unit 1)
 				)
@@
 		(dnp no)
 		(fields_autoplaced yes)
-		(property "Reference" "Fucked1"
+		(property "Reference" "U2"
 			(at 137.16 62.2299 0)
 			(effects
@@
 			(project ""
 				(path "/42dafeb3-7ab4-4fdc-a747-7ffb34623964"
-					(reference "Fucked1")
+					(reference "U2")
 					(unit 2)
 				)
