File: hardware/SignleCellBoard/SignleCellBoard.kicad_pcb (KiCad board)
At the start: 2 copper layers, 90 parts, among them J1 USB_C_Receptacle_USB2.0_14P, J10 Conn_01x02_Pin, J2 Conn_01x02_Pin, J3 Conn_01x02_Pin, J4 Conn_01x02_Pin, J5 Conn_01x02_Pin, J6 Conn_02x05_Odd_Even, J7 Conn_01x02_Pin, J8 Conn_01x02_Pin, J9 Barrel_Jack, SW1 SW_SPST, SW2 SW_SPST, U1 FT232RL, U10 TPS54202DDC, U11 TL071, U12 TL071, U2 LM7321MAX/NOPB, U3 STM32F091RCTx, U4 CD22M3494MQZ, U5 CD22M3494MQZ, U6 LM2776, U7 AD5263BRUZ200, U8 AD5263BRUZ200, U9 XTPS55285VALR

Commit message: Parker Loves Furries
Parts:
- removed C10, C30: 1µF, Capacitor_SMD:C_0603_1608Metric_Pad1.08x0.95mm_HandSolder
- removed C13, C14: 2.2u, Capacitor_SMD:C_0603_1608Metric_Pad1.08x0.95mm_HandSolder
- removed C15: 22u, SeniorDesign:CAP_EEFK_C_PAN
- removed C17: 1µF, Capacitor_SMD:C_0402_1005Metric_Pad0.74x0.62mm_HandSolder
- removed C18: 3.3µF, Capacitor_SMD:C_1210_3225Metric_Pad1.33x2.70mm_HandSolder
- removed C23: 56p, Capacitor_SMD:C_0201_0603Metric_Pad0.64x0.40mm_HandSolder
- removed C24, C25: 100nF, Capacitor_SMD:C_0402_1005Metric_Pad0.74x0.62mm_HandSolder
- removed C26: 1µF, Capacitor_SMD:C_0201_0603Metric_Pad0.64x0.40mm_HandSolder
- removed C27: 47u, Capacitor_SMD:C_0805_2012Metric_Pad1.18x1.45mm_HandSolder
- removed C28: 10µF, Capacitor_SMD:C_1210_3225Metric_Pad1.33x2.70mm_HandSolder
- removed C29: 33u, Capacitor_Tantalum_SMD:CP_EIA-3528-21_Kemet-B_HandSolder
- removed C31, C4, C5, C6, C8: 100nF, Capacitor_SMD:C_0603_1608Metric_Pad1.08x0.95mm_HandSolder
- removed C32, C9: 10nF, Capacitor_SMD:C_0603_1608Metric_Pad1.08x0.95mm_HandSolder
- removed C33: 1nF, Capacitor_SMD:C_0603_1608Metric_Pad1.08x0.95mm_HandSolder
- removed D3: BAT60JFILM, Diode_SMD:D_SOD-323_HandSoldering
- removed D4: BLUELED, Diode_SMD:D_0805_2012Metric_Pad1.15x1.40mm_HandSolder
- removed D5: REDLED, Diode_SMD:D_0805_2012Metric_Pad1.15x1.40mm_HandSolder
- removed D6: GREENLED, Diode_SMD:D_0805_2012Metric_Pad1.15x1.40mm_HandSolder
- removed D7, D8: 1N4148WT, Diode_SMD:D_SOD-123
- removed F4: 500mA, Fuse:Fuse_0603_1608Metric_Pad1.05x0.95mm_HandSolder
- removed FB1: 120R, Inductor_SMD:L_0603_1608Metric_Pad1.05x0.95mm_HandSolder
- removed J10: Conn_01x02_Pin, Connector_PinSocket_2.54mm:PinSocket_1x02_P2.54mm_Vertical
- removed L2: 10u, Inductor_SMD:L_Bourns_SRN6045TA
- removed R1, R10, R4, R9: 150Ω, Resistor_SMD:R_0603_1608Metric_Pad0.98x0.95mm_HandSolder
- removed R11: 24.9k, Resistor_SMD:R_0402_1005Metric_Pad0.72x0.64mm_HandSolder
- removed R12: 261k, Resistor_SMD:R_0402_1005Metric_Pad0.72x0.64mm_HandSolder
- removed R13, R15: 100k, Resistor_SMD:R_0402_1005Metric_Pad0.72x0.64mm_HandSolder
- removed R14: 8.87k, Resistor_SMD:R_0402_1005Metric_Pad0.72x0.64mm_HandSolder
- removed R16: 22.1k, Resistor_SMD:R_0402_1005Metric_Pad0.72x0.64mm_HandSolder
- removed R17: 6.04k, Resistor_SMD:R_0402_1005Metric_Pad0.72x0.64mm_HandSolder
- removed R2, R3: 10k, Resistor_SMD:R_0603_1608Metric_Pad0.98x0.95mm_HandSolder
- removed R7, R8: 10kΩ, Resistor_SMD:R_0603_1608Metric_Pad0.98x0.95mm_HandSolder
- removed Rfbt1: 102k, Resistor_SMD:R_0402_1005Metric_Pad0.72x0.64mm_HandSolder
- removed SW1, SW2: SW_SPST, Button_Switch_SMD:SW_SPST_SKQG_WithoutStem
- removed U11, U12: TL071, Package_SO:SOIC-8_3.9x4.9mm_P1.27mm
- removed U7: AD5263BRUZ200, SeniorDesign:SOP65P640X120-24N
- added JP1: SolderJumper_3_Open, Jumper:SolderJumper-3_P1.3mm_Open_Pad1.0x1.5mm, F.Cu at (205.7, 50.8)
- C1: value 100nF -> 1µF
- C11: value 1µF -> 100nF; footprint Capacitor_SMD:C_0603_1608Metric_Pad1.08x0.95mm_HandSolder -> Capacitor_SMD:C_0805_2012Metric_Pad1.18x1.45mm_HandSolder
- C12: value 1µF -> 56p; footprint Capacitor_SMD:C_0603_1608Metric_Pad1.08x0.95mm_HandSolder -> Capacitor_SMD:C_0603_1608Metric
- C16: value 4.7u -> 47u; footprint Capacitor_SMD:C_1210_3225Metric_Pad1.33x2.70mm_HandSolder -> Capacitor_SMD:C_0805_2012Metric_Pad1.18x1.45mm_HandSolder
- C19: value 240p -> 1µF; footprint Capacitor_SMD:C_0402_1005Metric_Pad0.74x0.62mm_HandSolder -> Capacitor_SMD:C_0603_1608Metric_Pad1.08x0.95mm_HandSolder; moved to B.Cu
- C2, C3: value 10µF -> 2.2u
- C20: value 4.7u -> 100nF; footprint Capacitor_SMD:C_0201_0603Metric_Pad0.64x0.40mm_HandSolder -> Capacitor_SMD:C_0603_1608Metric_Pad1.08x0.95mm_HandSolder
- C21: value 15n -> 10nF; footprint Capacitor_SMD:C_0402_1005Metric_Pad0.74x0.62mm_HandSolder -> Capacitor_SMD:C_0603_1608Metric_Pad1.08x0.95mm_HandSolder; moved to B.Cu
- C22: value 100nF -> 1nF; footprint Capacitor_SMD:C_0805_2012Metric_Pad1.18x1.45mm_HandSolder -> Capacitor_SMD:C_0603_1608Metric_Pad1.08x0.95mm_HandSolder; moved to B.Cu
- C7: value 100nF -> 3.3µF; footprint Capacitor_SMD:C_0603_1608Metric_Pad1.08x0.95mm_HandSolder -> Capacitor_SMD:C_1210_3225Metric_Pad1.33x2.70mm_HandSolder
- D1: value REDLED -> 1N4148WT; footprint Diode_SMD:D_0805_2012Metric_Pad1.15x1.40mm_HandSolder -> Diode_SMD:D_SOD-123; moved to B.Cu
- D2: value GREENLED -> 1N4148WT; footprint Diode_SMD:D_0805_2012Metric_Pad1.15x1.40mm_HandSolder -> Diode_SMD:D_SOD-123
- J1: value USB_C_Receptacle_USB2.0_14P -> Conn_01x02_Pin; footprint Connector_USB:USB_C_Receptacle_G-Switch_GT-USB-7010ASV -> Connector_PinSocket_2.54mm:PinSocket_1x02_P2.54mm_Vertical
- J5: value Conn_01x02_Pin -> Conn_01x30_Pin; footprint Connector_PinSocket_2.54mm:PinSocket_1x02_P2.54mm_Vertical -> Connector_PinSocket_2.54mm:PinSocket_1x30_P2.54mm_Vertical
- J6: value Conn_02x05_Odd_Even -> Conn_01x30_Pin; footprint Connector_PinHeader_2.54mm:PinHeader_2x05_P2.54mm_Vertical -> Connector_PinSocket_2.54mm:PinSocket_1x30_P2.54mm_Vertical
- J7: value Conn_01x02_Pin -> Conn_01x06_Socket; footprint Connector_PinSocket_2.54mm:PinSocket_1x02_P2.54mm_Vertical -> Connector_PinSocket_2.54mm:PinSocket_1x06_P2.54mm_Vertical
- J8: value Conn_01x02_Pin -> Barrel_Jack; footprint Connector_PinSocket_2.54mm:PinSocket_1x02_P2.54mm_Vertical -> Connector_BarrelJack:BarrelJack_CUI_PJ-063AH_Horizontal
- J9: value Barrel_Jack -> Conn_01x02_Pin; footprint Connector_BarrelJack:BarrelJack_CUI_PJ-063AH_Horizontal -> Connector_PinSocket_2.54mm:PinSocket_1x02_P2.54mm_Vertical
- R5: value 150Ω -> 100k; footprint Resistor_SMD:R_0603_1608Metric_Pad0.98x0.95mm_HandSolder -> Resistor_SMD:R_0402_1005Metric_Pad0.72x0.64mm_HandSolder
- R6: value 10kΩ -> 22.1k; footprint Resistor_SMD:R_0603_1608Metric_Pad0.98x0.95mm_HandSolder -> Resistor_SMD:R_0402_1005Metric_Pad0.72x0.64mm_HandSolder
- U1: value FT232RL -> DIP; footprint Package_SO:SSOP-28_5.3x10.2mm_P0.65mm -> Package_DIP:DIP-40_W15.24mm
- U10: value TPS54202DDC -> TL071; footprint Package_TO_SOT_SMD:SOT-23-6 -> Package_SO:SOIC-8_3.9x4.9mm_P1.27mm; moved to B.Cu
- U2: value LM7321MAX/NOPB -> DIP; footprint Package_SO:SOIC-8_3.9x4.9mm_P1.27mm -> Package_DIP:DIP-40_W15.24mm
- U3: value STM32F091RCTx -> LM7321MAX/NOPB; footprint Package_QFP:LQFP-64_10x10mm_P0.5mm -> Package_SO:SOIC-8_3.9x4.9mm_P1.27mm
- U4: value CD22M3494MQZ -> AD5263BRUZ200; footprint SeniorDesign:PLCC44_16P66X16P66_INR-M -> Package_DIP:DIP-24_W15.24mm
- U5: value CD22M3494MQZ -> LM2776; footprint SeniorDesign:PLCC44_16P66X16P66_INR-M -> Package_TO_SOT_SMD:SOT-23-6
- U6: value LM2776 -> AD5263BRUZ200; footprint Package_TO_SOT_SMD:SOT-23-6 -> Package_DIP:DIP-24_W15.24mm
- U8: value AD5263BRUZ200 -> TPS54202DDC; footprint SeniorDesign:SOP65P640X120-24N -> Package_TO_SOT_SMD:SOT-23-6
- U9: value XTPS55285VALR -> TL071; footprint SeniorDesign:TPS55285 -> Package_SO:SOIC-8_3.9x4.9mm_P1.27mm; moved to B.Cu
- moved C19 237.1 mm to (261.6, 82.5), turned to 90 degrees
- moved C21 236.1 mm to (261.6, 92.7)
- moved C16 219.4 mm to (235.3, 26.4), turned to 180 degrees
- moved C22 214.4 mm to (261.6, 77.9), turned to -90 degrees
- moved U9 213.4 mm to (233.7, 122.6), turned to 180 degrees
- moved L1 204.1 mm to (227.2, 36.5), turned to 180 degrees
- moved U10 188.4 mm to (248.9, 122.6)
- moved C20 186.7 mm to (250.6, 110.5), turned to 180 degrees
- moved J9 181.8 mm to (228.6, 134.6), turned to 90 degrees
- moved C12 176.6 mm to (227.4, 30.3), turned to 90 degrees
- moved F3 175.8 mm to (206.6, 54.6), turned to -90 degrees
- moved F2 164.3 mm to (217.6, 29.2), turned to 0 degrees
- moved D1 149.8 mm to (261.6, 87.6), turned to 90 degrees
- moved U6 149.4 mm to (242.6, 85.1)
- moved J3 133.0 mm to (261.6, 134.6), turned to -90 degrees
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Connections:
- C1 pad 1: Net-(U1-3V3OUT) -> Net-(U5-C1-)
- C1 pad 2: GND -> Net-(U5-C1+)
- C11 pad 1: +3.3V -> Net-(U8-BOOT)
- C11 pad 2: GND -> Net-(U8-SW)
- C12 pad 1: Net-(U6-C1-) -> Net-(U8-FB)
- C12 pad 2: Net-(U6-C1+) -> Net-(C12-Pad2)
- C16 pad 1: /WallAdpt -> GND
- C16 pad 2: GND -> Net-(C12-Pad2)
- C19 pad 1: Net-(U9-COMP) -> /Standard_Cell/C1_in
- C19 pad 2: GND -> /Standard_Cell/C1_out
- C2 pad 1: +3.3V -> GND
- C2 pad 2: GND -> +5V
- C20 pad 1: Net-(U9-VCC) -> /Standard_Cell/C2_in
- C20 pad 2: GND -> /Standard_Cell/C2_out
- C21 pad 1: Net-(C21-Pad1) -> /Standard_Cell/C3_in
- C21 pad 2: GND -> /Standard_Cell/C3_out
- C22 pad 1: Net-(U10-BOOT) -> /Standard_Cell/C4_in
- C22 pad 2: Net-(U10-SW) -> /Standard_Cell/C4_out
- C3 pad 1: Net-(D3-K) -> GND
- C3 pad 2: GND -> Net-(U5-VOUT)
- C7 pad 1: +3.3V -> GND
- C7 pad 2: GND -> +5V
- D1 pad 1: /LED_TX -> /Standard_Cell/D1_cathode
- D1 pad 2: Net-(D1-A) -> /Standard_Cell/D1_anode
- D2 pad 1: /LED_RX -> /Standard_Cell/D2_cathode
- D2 pad 2: Net-(D2-A) -> /Standard_Cell/D2_anode
- F1 pad 1: Net-(F1-Pad1) -> -5V
- F1 pad 2: Net-(D3-A) -> Net-(U5-VOUT)
- F2 pad 1: -5V -> +3.3V
- F2 pad 2: Net-(U6-VOUT) -> Net-(C12-Pad2)
- F3 pad 1: +3.3V -> Net-(JP1-C)
- F3 pad 2: Net-(C23-Pad2) -> +5V
- J2 pad 1: /Standard_Cell/Y0 -> /Standard_Cell/Y1
- J3 pad 1: /Standard_Cell/Y1 -> /Standard_Cell/Y2
- J4 pad 1: /Standard_Cell/Y2 -> GND
- J4 pad 2: GND -> Net-(J4-Pin_2)
- J5 pad 2: Net-(J5-Pin_2) -> /MT_STB
- J6 pad 1: /NRST -> +5V
- J6 pad 10: unconnected-(J6-Pin_10-Pad10) -> /BRUZ_NRST
- J6 pad 2: /SWDIO -> unconnected-(J6-Pin_2-Pad2)
- J6 pad 4: GND -> /PD2
- J6 pad 6: /SWCLK -> unconnected-(J6-Pin_6-Pad6)
- J6 pad 7: +3.3V -> unconnected-(J6-Pin_7-Pad7)
- J6 pad 8: +3.3V -> unconnected-(J6-Pin_8-Pad8)
- J7 pad 1: /PC3 -> unconnected-(J7-Pin_1-Pad1)
- J7 pad 2: /PC2 -> /PC12
- J8 pad 1: /XOSC_OUT -> /WallAdpt
- J8 pad 2: /XOSC_IN -> GND
- J9 pad 1: /WallAdpt -> /Standard_Cell/J1_out
- J9 pad 2: GND -> /Standard_Cell/J1_in
- L1 pad 1: Net-(U10-SW) -> Net-(U8-SW)
- L1 pad 2: Net-(C23-Pad2) -> Net-(C12-Pad2)
- R5 pad 1: /LED_STM_1 -> Net-(C12-Pad2)
- R5 pad 2: Net-(D4-A) -> Net-(U8-FB)
- R6 pad 1: Net-(SW2-B) -> Net-(U8-FB)
- U1 pad 1: Net-(U1-TXD) -> /Standard_Cell/Y3
- U1 pad 10: unconnected-(U1-DCD-Pad10) -> /Standard_Cell/R2_in
- U1 pad 11: Net-(U1-CTS) -> /Standard_Cell/R2_out
- U1 pad 12: unconnected-(U1-CBUS4-Pad12) -> /Standard_Cell/R4_in
- U1 pad 13: unconnected-(U1-CBUS2-Pad13) -> /Standard_Cell/R4_out
- U1 pad 14: unconnected-(U1-CBUS3-Pad14) -> (no net)
- U1 pad 15: Net-(U1-USBD+) -> /Standard_Cell/Y7
- U1 pad 16: Net-(U1-USBD-) -> GND
- U1 pad 17: Net-(U1-3V3OUT) -> /Standard_Cell/Y6
- U1 pad 18: GND -> /MT_STB
- U1 pad 19: unconnected-(U1-~{RESET}-Pad19) -> /Standard_Cell/Y5
- U1 pad 2: unconnected-(U1-DTR-Pad2) -> /MT_AY2
- U1 pad 20: Net-(D3-K) -> -5V
- U1 pad 22: /LED_RX -> /MT_AX1
- U1 pad 23: /LED_TX -> /MT_AX2
- U1 pad 24: (no net) -> /MT_AY0
- U1 pad 25: GND -> /MT_AY1
- U1 pad 26: GND -> /Standard_Cell/J1_out
- U1 pad 27: unconnected-(U1-OSCI-Pad27) -> /Standard_Cell/J1_in
- U1 pad 28: unconnected-(U1-OSCO-Pad28) -> /Standard_Cell/Op1_out
- U1 pad 3: unconnected-(U1-RTS-Pad3) -> /MT_RST
- U1 pad 4: +3.3V -> /MT_AX3
- U1 pad 5: Net-(U1-RXD) -> /MT_AX0
- U1 pad 6: unconnected-(U1-RI-Pad6) -> /Standard_Cell/C2_in
- U1 pad 7: GND -> /Standard_Cell/C2_out
- U1 pad 8: (no net) -> /Standard_Cell/D2_cathode
- U1 pad 9: unconnected-(U1-DCR-Pad9) -> /Standard_Cell/D2_anode
- U10 pad 1: GND -> unconnected-(U10-NULL-Pad1)
- U10 pad 2: Net-(U10-SW) -> /Standard_Cell/Op2_neg
- U10 pad 3: /WallAdpt -> /Standard_Cell/Op2_pos
- U10 pad 4: Net-(U10-FB) -> -5V
- U10 pad 6: Net-(U10-BOOT) -> /Standard_Cell/Op2_out
- U2 pad 1: unconnected-(U2-NULL-Pad1) -> /Standard_Cell/Y3
- U2 pad 2: Net-(J5-Pin_2) -> /MT_AY2
- U2 pad 3: /Standard_Cell/Y3 -> /MT_RST
- U2 pad 4: -5V -> /MT_AX3
- U2 pad 5: unconnected-(U2-NULL-Pad5) -> /MT_AX0
- U2 pad 6: Net-(J5-Pin_2) -> /Standard_Cell/C3_out
- U2 pad 7: +5V -> /Standard_Cell/C3_in
- U2 pad 8: unconnected-(U2-NC-Pad8) -> /Standard_Cell/D1_cathode
- U3 pad 1: +3.3V -> unconnected-(U3-NULL-Pad1)
- U3 pad 2: unconnected-(U3-PC13-Pad2) -> Net-(J4-Pin_2)
- U3 pad 3: /XOSC_IN -> /Standard_Cell/Y3
- U3 pad 4: /XOSC_OUT -> -5V
- U3 pad 6: unconnected-(U3-PF1-Pad6) -> Net-(J4-Pin_2)
- U3 pad 7: /NRST -> +5V
- U4 pad 1: (no net) -> /Standard_Cell/R5_in
- U4 pad 10: /Standard_Cell/Y7 -> +5V
- U4 pad 11: (no net) -> /PA7
- U4 pad 12: GND -> /PA5
- U4 pad 13: /Standard_Cell/Y6 -> /BRUZ_NCS_1
- U4 pad 14: /MT_STB -> /BRUZ_NRST
- U4 pad 15: /Standard_Cell/Y5 -> +5V
- U4 pad 16: -5V -> unconnected-(U4A-SDO/O1-Pad16)
- U4 pad 17: GND -> unconnected-(U4A-NC/O2-Pad17)
- U4 pad 18: /MT_AX1 -> -5V
- U4 pad 19: /MT_AX2 -> unconnected-(U4E-W4-Pad19)
- U4 pad 2: /Standard_Cell/C2_in -> /Standard_Cell/R5_out
- U4 pad 20: /MT_AY0 -> unconnected-(U4E-A4-Pad20)
- U4 pad 21: /MT_AY1 -> unconnected-(U4E-B4-Pad21)
- U4 pad 22: (no net) -> unconnected-(U4C-W2-Pad22)
- U4 pad 23: (no net) -> unconnected-(U4C-A2-Pad23)
- U4 pad 24: /Standard_Cell/D2_anode -> unconnected-(U4C-B2-Pad24)
- U4 pad 3: /Standard_Cell/C2_out -> /Standard_Cell/R5_out
- U4 pad 4: /Standard_Cell/D1_cathode -> /Standard_Cell/R6_in
- U4 pad 5: /Standard_Cell/D1_anode -> /Standard_Cell/R6_out
- U4 pad 6: /Standard_Cell/C4_in -> /Standard_Cell/R6_out
- U4 pad 7: /Standard_Cell/C4_out -> +5V
- U4 pad 8: /Standard_Cell/C3_in -> GND
- U4 pad 9: /Standard_Cell/C3_out -> GND
- U5 pad 1: (no net) -> Net-(U5-VOUT)
- U5 pad 2: /Standard_Cell/R3_out -> GND
- U5 pad 3: /Standard_Cell/R3_in -> +5V
- U5 pad 4: /Standard_Cell/R1_out -> +5V
- U5 pad 5: /Standard_Cell/R1_in -> Net-(U5-C1+)
- U5 pad 6: /Standard_Cell/R2_in -> Net-(U5-C1-)
- U6 pad 1: Net-(U6-VOUT) -> /Standard_Cell/R1_in
- U6 pad 2: GND -> /Standard_Cell/R1_out
- U6 pad 3: +5V -> /Standard_Cell/R1_out
- U6 pad 4: unconnected-(U6-EN-Pad4) -> /Standard_Cell/R3_in
- U6 pad 5: Net-(U6-C1+) -> /Standard_Cell/R3_out
- U6 pad 6: Net-(U6-C1-) -> /Standard_Cell/R3_out
- U8 pad 1: /Standard_Cell/R5_in -> GND
- U8 pad 2: /Standard_Cell/R5_out -> Net-(U8-SW)
- U8 pad 3: /Standard_Cell/R5_out -> +5V
- U8 pad 4: /Standard_Cell/R6_in -> Net-(U8-FB)
- U8 pad 5: /Standard_Cell/R6_out -> unconnected-(U8-EN-Pad5)
- U8 pad 6: /Standard_Cell/R6_out -> Net-(U8-BOOT)
- U9 pad 1: Net-(U9-MODE) -> unconnected-(U9-NULL-Pad1)
- U9 pad 2: unconnected-(U9-SCL-Pad2) -> /Standard_Cell/Op1_neg
- U9 pad 3: unconnected-(U9-SDA-Pad3) -> /Standard_Cell/Op1_pos
- U9 pad 4: Net-(U9-EN_UVLO) -> -5V
- U9 pad 5: /WallAdpt -> unconnected-(U9-NULL-Pad5)
- U9 pad 6: Net-(U9-SW1) -> /Standard_Cell/Op1_out
- U9 pad 7: GND -> +5V
- U9 pad 8: Net-(U9-SW2) -> unconnected-(U9-NC-Pad8)
Routing:
- net GND: track 13.7 -> 350.6 mm, vias 0 -> 2
- net +5V: track 0.00 -> 255.4 mm, vias 0 -> 1
- net -5V: track 0.00 -> 177.6 mm, vias 0 -> 2
- net /MT_AX1: track 0.00 -> 120.7 mm
- net /MT_AX2: track 0.00 -> 119.2 mm
- net /MT_AY0: track 0.00 -> 117.7 mm
- net /MT_AY1: track 0.00 -> 116.6 mm
- net /MT_STB: track 0.00 -> 87.1 mm, vias 0 -> 1
- net /Standard_Cell/Y7: track 0.00 -> 81.4 mm
- net /Standard_Cell/Y2: track 0.00 -> 79.4 mm
- net /Standard_Cell/Y1: track 0.00 -> 77.0 mm
- net /Standard_Cell/Y0: track 0.00 -> 76.0 mm
- net /Standard_Cell/Y3: track 0.00 -> 67.6 mm
- net /MT_DAT: track 0.00 -> 63.4 mm
- net /MT_AX0: track 0.00 -> 50.2 mm
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
Commit message: I know of at least one
Parts:
- C1, C11, C2, R6: moved to B.Cu
- C7: footprint Capacitor_SMD:C_1210_3225Metric_Pad1.33x2.70mm_HandSolder -> Capacitor_SMD:C_0805_2012Metric_Pad1.18x1.45mm_HandSolder
- JP1: footprint Jumper:SolderJumper-3_P1.3mm_Open_Pad1.0x1.5mm -> Jumper:SolderJumper-3_P1.3mm_Open_Pad1.0x1.5mm_NumberLabels
- U5, U8: footprint Package_TO_SOT_SMD:SOT-23-6 -> Connector_PinHeader_2.54mm:PinHeader_1x06_P2.54mm_Vertical
- moved F2 28.4 mm to (222.6, 57.1)
- moved R6 21.9 mm to (232.4, 50.8)
- moved C7 20.6 mm to (237.2, 50.8), turned to 180 degrees
- moved C16 19.8 mm to (243.8, 44.2), turned to 90 degrees
- moved J5 19.0 mm to (184.2, 132.1)
- moved U5 17.7 mm to (260.4, 39.4), turned to -90 degrees
- moved J6 16.5 mm to (201.9, 58.4)
- moved U8 15.2 mm to (240.0, 47.0), turned to -90 degrees
- moved C12 14.3 mm to (235.7, 41.9), turned to 0 degrees
- moved R5 13.6 mm to (235.5, 39.4)
- moved L1 13.3 mm to (240.0, 40.3), turned to 90 degrees
- moved C3 12.6 mm to (259.1, 43.2), turned to 0 degrees
- moved J7 12.5 mm to (186.7, 39.3), turned to 90 degrees
- moved C11 12.3 mm to (228.8, 43.2), turned to 0 degrees
- moved C1 9.61 mm to (248.5, 43.2), turned to 0 degrees
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Connections:
- J5 pad 2: /MT_STB -> /MT_AX1
- J5 pad 3: /MT_RST -> /MT_AX2
- J5 pad 4: /BRUZ_NCS_1 -> /PB5
- J5 pad 5: /BRUZ_NCS_0 -> /PB4
- J5 pad 6: /MT_CS_1 -> /MT_AY0
- J5 pad 7: /MT_CS_0 -> unconnected-(J5-Pin_7-Pad7)
- J6 pad 16: unconnected-(J6-Pin_16-Pad16) -> /BRUZ_NCS_1
- J6 pad 17: unconnected-(J6-Pin_17-Pad17) -> /BRUZ_NRST
- J6 pad 18: unconnected-(J6-Pin_18-Pad18) -> /BRUZ_NCS_0
- J6 pad 19: unconnected-(J6-Pin_19-Pad19) -> /MT_CS_0
- J6 pad 20: unconnected-(J6-Pin_20-Pad20) -> /MT_DAT
- J6 pad 22: /MT_AX3 -> /MT_STB
- J6 pad 23: /MT_AX2 -> /MT_AX0
- J6 pad 24: /MT_AX1 -> /MT_AX3
- J6 pad 25: /MT_AX0 -> /MT_RST
- J6 pad 27: /MT_AY1 -> /MT_DAT
- J6 pad 28: /MT_AY0 -> /MT_CS_1
- J6 pad 29: /MT_DAT -> /MT_AY1
Routing:
- net GND: track 350.6 -> 530.7 mm
- net +5V: track 255.4 -> 397.8 mm
- net +3.3V: track 0.00 -> 86.0 mm, vias 0 -> 1
- net /MT_DAT: track 63.4 -> 132.4 mm, vias 0 -> 1
- net /PC12: track 0.00 -> 61.8 mm
- net /MT_AY0: track 117.7 -> 167.6 mm
- net /MT_AX3: track 30.7 -> 75.6 mm
- net /MT_AX2: track 119.2 -> 163.4 mm
- net /MT_RST: track 31.4 -> 74.6 mm
- net /MT_AY2: track 33.4 -> 74.6 mm
- net /MT_AX1: track 120.7 -> 161.7 mm
- net /PA7: track 25.9 -> 64.4 mm
- net /PA5: track 24.2 -> 60.9 mm
- net /PD2: track 0.00 -> 30.9 mm
- net /MT_AY1: track 116.6 -> 143.9 mm
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Other:
- board outline added: 95.2 x 105.4 mm

Commit message: feat: WIP on manufacturability
Parts:
- moved F2 0.98 mm to (223.6, 57.1)
Routing:
- net /Standard_Cell/R6_out: track 26.9 -> 29.1 mm
- net Net-(C12-Pad2): track 48.1 -> 46.8 mm
- net +3.3V: track 86.0 -> 87.0 mm
- net -5V: track 183.3 -> 184.0 mm
Changed lines of the file:
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@@
 		(tags "744773112 ")
 		(property "Reference" "L1"
-			(at 0.858975 0.9825 90)
+			(at 3.0352 3.07 90)
 			(unlocked yes)
 			(layer "F.SilkS")
@@
 	(footprint "Fuse:Fuse_0603_1608Metric_Pad1.05x0.95mm_HandSolder"
 		(layer "F.Cu")
-		(at 222.645 57.15)
+		(at 223.625 57.15)
 		(descr "Fuse SMD 0603 (1608 Metric), square (rectangular) end terminal, IPC-7351 nominal with elongated pad for handsoldering. (Body size source: http://www.tortai-tech.com/upload/download/2011102023233369053.pdf), generated with kicad-footprint-generator")
 		(tags "fuse handsolder")
@@
 	)
 	(segment
+		(start 242.961393 60.5)
+		(end 243.84 59.621393)
+		(width 0.8)
+		(layer "F.Cu")
+		(net 1)
+	)
+	(segment
 		(start 261.62 68.58)
 		(end 254 60.96)
@@
 	)
 	(segment
-		(start 240.03 46.99)
-		(end 241.765 45.255)
+		(start 243.84 59.621393)
+		(end 243.84 55.88)
 		(width 0.8)
 		(layer "F.Cu")
@@
 	)
 	(segment
-		(start 222.25 64.77)
-		(end 224.79 62.23)
+		(start 240.03 46.99)
+		(end 241.765 45.255)
 		(width 0.8)
 		(layer "F.Cu")
@@
 	)
 	(segment
-		(start 243.84 59.621393)
-		(end 243.84 55.88)
-		(width 0.8)
-		(layer "F.Cu")
-		(net 1)
-	)
-	(segment
 		(start 238.76 50.8)
 		(end 240.03 49.53)
@@
 	)
 	(segment
-		(start 241.231393 62.23)
-		(end 243.84 59.621393)
+		(start 232.41 93.98)
+		(end 224.79 86.36)
 		(width 0.8)
 		(layer "F.Cu")
@@
 	)
 	(segment
-		(start 232.41 93.98)
-		(end 224.79 86.36)
+		(start 240.03 49.53)
+		(end 240.03 46.99)
 		(width 0.8)
 		(layer "F.Cu")
@@
 	)
 	(segment
-		(start 240.03 49.53)
-		(end 240.03 46.99)
+		(start 226.52 60.5)
+		(end 242.961393 60.5)
 		(width 0.8)
 		(layer "F.Cu")
@@
 	)
 	(segment
-		(start 224.79 62.23)
-		(end 241.231393 62.23)
+		(start 222.25 64.77)
+		(end 226.52 60.5)
 		(width 0.8)
 		(layer "F.Cu")
@@
 	(via
 		(at 254 52.07)
-		(size 0.7)
-		(drill 0.3)
+		(size 1.2)
+		(drill 0.7)
 		(layers "F.Cu" "B.Cu")
 		(net 1)
@@
 	(via
 		(at 243.84 55.88)
-		(size 0.7)
-		(drill 0.3)
+		(size 1.2)
+		(drill 0.7)
 		(layers "F.Cu" "B.Cu")
 		(net 1)
@@
 	)
 	(segment
-		(start 221.77 57.15)
+		(start 222.75 57.15)
 		(end 219.71 57.15)
 		(width 0.4)
@@
 	(via
 		(at 219.71 57.15)
-		(size 0.7)
-		(drill 0.3)
+		(size 1.2)
+		(drill 0.7)
 		(layers "F.Cu" "B.Cu")
 		(net 2)
@@
 	(via
 		(at 255.27 123.19)
-		(size 0.7)
-		(drill 0.3)
+		(size 1.2)
+		(drill 0.7)
 		(layers "F.Cu" "B.Cu")
 		(net 5)
 	)
 	(segment
-		(start 219.71 100.33)
-		(end 219.71 101.6)
+		(start 219.71 100.39)
+		(end 213.36 106.74)
 		(width 0.6)
 		(layer "B.Cu")
@@
 	)
 	(segment
-		(start 213.36 107.95)
-		(end 213.36 114.3)
+		(start 255.27 123.19)
+		(end 251.395 123.19)
 		(width 0.6)
 		(layer "B.Cu")
@@
 	)
 	(segment
-		(start 219.71 101.6)
-		(end 213.36 107.95)
+		(start 213.36 114.3)
+		(end 220.98 121.92)
 		(width 0.6)
 		(layer "B.Cu")
@@
 	)
 	(segment
-		(start 255.27 123.19)
-		(end 251.395 123.19)
+		(start 213.36 106.74)
+		(end 213.36 114.3)
 		(width 0.6)
 		(layer "B.Cu")
@@
 	)
 	(segment
-		(start 213.36 114.3)
-		(end 220.98 121.92)
-		(width 0.6)
+		(start 255.6775 43.18)
+		(end 255.6775 39.7775)
+		(width 0.4)
 		(layer "B.Cu")
 		(net 5)
 	)
 	(segment
-		(start 255.6775 43.18)
-		(end 255.6775 39.7775)
-		(width 0.4)
+		(start 219.71 100.33)
+		(end 219.71 100.39)
+		(width 0.6)
 		(layer "B.Cu")
 		(net 5)
@@
 	)
 	(segment
+		(start 245.11 43.18)
+		(end 246.38 44.45)
+		(width 0.6)
+		(layer "F.Cu")
+		(net 10)
+	)
+	(segment
 		(start 236.5 40.92)
 		(end 236.22 40.64)
@@
 	)
 	(segment
-		(start 246.38 44.45)
-		(end 246.38 48.26)
-		(width 0.6)
-		(layer "F.Cu")
-		(net 10)
-	)
-	(segment
 		(start 243.84 43.18)
 		(end 243.84 39.37)
@@
 	)
 	(segment
-		(start 243.84 43.18)
-		(end 245.11 43.18)
-		(width 0.6)
-		(layer "F.Cu")
-		(net 10)
-	)
-	(segment
-		(start 237.49 57.15)
-		(end 223.52 57.15)
+		(start 236.7546 38.7604)
+		(end 236.145 39.37)
 		(width 0.6)
 		(layer "F.Cu")
@@
 	)
 	(segment
-		(start 236.7546 38.7604)
-		(end 236.145 39.37)
+		(start 243.84 39.37)
+		(end 243.2304 38.7604)
 		(width 0.6)
 		(layer "F.Cu")
@@
 	)
 	(segment
-		(start 243.84 39.37)
-		(end 243.2304 38.7604)
+		(start 246.38 44.45)
+		(end 246.38 48.26)
 		(width 0.6)
 		(layer "F.Cu")
@@
 	)
 	(segment
-		(start 245.11 43.18)
-		(end 246.38 44.45)
+		(start 237.49 57.15)
+		(end 224.8 57.15)
 		(width 0.6)
 		(layer "F.Cu")
@@
 	)
 	(segment
+		(start 243.84 43.18)
+		(end 245.11 43.18)
+		(width 0.6)
+		(layer "F.Cu")
+		(net 10)
+	)
+	(segment
 		(start 236.22 39.445)
 		(end 236.145 39.37)
@@
 	(via
 		(at 246.38 68.58)
-		(size 0.7)
-		(drill 0.3)
+		(size 1.2)
+		(drill 0.7)
 		(layers "F.Cu" "B.Cu")
 		(net 24)
@@
 	(via
 		(at 250.19 54.61)
-		(size 0.7)
-		(drill 0.3)
+		(size 1.2)
+		(drill 0.7)
 		(layers "F.Cu" "B.Cu")
 		(net 24)
 	)
 	(segment
-		(start 220.98 102.87)
-		(end 224.79 102.87)
-		(width 0.6)
-		(layer "B.Cu")
-		(net 24)
-	)
-	(segment
 		(start 246.38 96.52)
 		(end 245.11 97.79)
@@
 	)
 	(segment
+		(start 215.9 114.3)
+		(end 215.9 106.7)
+		(width 0.6)
+		(layer "B.Cu")
+		(net 24)
+	)
+	(segment
 		(start 236.155 124.46)
 		(end 234.95 124.46)
@@
 	)
 	(segment
-		(start 215.9 114.3)
-		(end 215.9 107.95)
+		(start 220.3 102.3)
+		(end 225.36 102.3)
 		(width 0.6)
 		(layer "B.Cu")
@@
 	)
 	(segment
-		(start 215.9 107.95)
-		(end 220.98 102.87)
-		(width 0.6)
-		(layer "B.Cu")
-		(net 24)
-	)
-	(segment
 		(start 234.95 124.46)
 		(end 233.68 123.19)
@@
 	)
 	(segment
-		(start 254 58.42)
-		(end 265.43 58.42)
+		(start 215.9 106.7)
+		(end 220.3 102.3)
 		(width 0.6)
 		(layer "B.Cu")
@@
 	)
 	(segment
-		(start 246.445 120.65)
-		(end 246.445 118.175)
+		(start 225.36 102.3)
+		(end 227.33 100.33)
 		(width 0.6)
 		(layer "B.Cu")
@@
 	)
 	(segment
-		(start 224.79 102.87)
-		(end 227.33 100.33)
+		(start 254 58.42)
+		(end 265.43 58.42)
+		(width 0.6)
+		(layer "B.Cu")
+		(net 24)
+	)
+	(segment
+		(start 246.445 120.65)
+		(end 246.445 118.175)
 		(width 0.6)
 		(layer "B.Cu")
@@
 	(via
 		(at 224.79 106.68)
-		(size 0.7)
-		(drill 0.3)
+		(size 1.2)
+		(drill 0.7)
 		(layers "F.Cu" "B.Cu")
 		(net 40)
@@
 	(via
 		(at 222.25 104.14)
-		(size 0.7)
-		(drill 0.3)
+		(size 1.2)
+		(drill 0.7)
 		(layers "F.Cu" "B.Cu")
 		(net 47)
@@
 	(via
 		(at 231.14 111.76)
-		(size 0.7)
-		(drill 0.3)
+		(size 1.2)
+		(drill 0.7)
 		(layers "F.Cu" "B.Cu")
 		(net 52)
@@
 	)
 	(segment
+		(start 232.41 62.51)
+		(end 232.4 62.5)
+		(width 0.4)
+		(layer "F.Cu")
+		(net 54)
+	)
+	(segment
 		(start 232.41 66.04)
 		(end 232.41 64.77)
@@
 		(width 0.4)
 		(layer "F.Cu")
+		(net 54)
+	)
+	(segment
+		(start 232.41 64.77)
+		(end 232.41 62.51)
+		(width 0.4)
+		(layer "F.Cu")

Commit message: PCB done
Parts:
- U1, U2: footprint Package_DIP:DIP-40_W15.24mm -> Package_DIP:DIP-40_W15.24mm_LongPads
- U5, U8: footprint Connector_PinHeader_2.54mm:PinHeader_1x06_P2.54mm_Vertical -> Connector_PinSocket_2.54mm:PinSocket_1x06_P2.54mm_Vertical
- moved F2 1.27 mm to (223.6, 55.9)
Routing:
- net GND: track 530.7 -> 533.5 mm
- net /Standard_Cell/R6_out: track 29.1 -> 26.9 mm
- net +5V: track 397.8 -> 399.7 mm
- net -5V: track 184.0 -> 185.6 mm
- net /Standard_Cell/Y3: track 67.6 -> 69.1 mm
- net /PA7: track 64.4 -> 63.0 mm
- net +3.3V: track 87.0 -> 88.2 mm
- net /MT_STB: track 108.3 -> 107.2 mm
- net /Standard_Cell/Y7: track 81.4 -> 82.4 mm
- net /MT_DAT: track 132.4 -> 133.4 mm
- net /Standard_Cell/Y0: track 76.0 -> 76.8 mm
- net /MT_RST: track 74.6 -> 75.3 mm
- net /PD2: track 30.9 -> 31.7 mm
- net /MT_AY2: track 74.6 -> 75.3 mm
- net /MT_AX3: track 75.6 -> 76.4 mm
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