File: hardware/SignleCellBoard/SignleCellBoard.kicad_sch (KiCad schematic)
At the start: 81 parts, among them J1 USB_C_Receptacle_USB2.0_14P, J2 Conn_01x02_Pin, J3 Conn_01x02_Pin, J4 Conn_01x02_Pin, J5 Conn_01x02_Pin, J6 Conn_02x05_Odd_Even, J7 Conn_01x02_Pin, J8 Conn_01x02_Pin, J9 Barrel_Jack, SW1 SW_SPST, SW2 SW_SPST, U1 FT232RL, U10 TPS54202DDC, U2 LM7321MAX/NOPB, U3 STM32F091RCTx, U4 CD22M3494MQZ, U5 CD22M3494MQZ, U6 LM2776, U7 AD5263BRUZ200, U8 AD5263BRUZ200, U9 XTPS55285VALR

Commit message: AAAAAAAAH
Parts:
- removed C1, C4, C5, C6, C7, C8: 100nF, Capacitor_SMD:C_0603_1608Metric_Pad1.08x0.95mm_HandSolder, symbol Device:C
- removed C10, C11: 1µF, Capacitor_SMD:C_0603_1608Metric_Pad1.08x0.95mm_HandSolder, symbol Device:C
- removed C2, C3: 10µF, Capacitor_SMD:C_0603_1608Metric_Pad1.08x0.95mm_HandSolder, symbol Device:C
- removed C9: 10nF, Capacitor_SMD:C_0603_1608Metric_Pad1.08x0.95mm_HandSolder, symbol Device:C
- removed D1, D5: REDLED, Diode_SMD:D_0805_2012Metric_Pad1.15x1.40mm_HandSolder, symbol Device:LED
- removed D2, D6: GREENLED, Diode_SMD:D_0805_2012Metric_Pad1.15x1.40mm_HandSolder, symbol Device:LED
- removed D3: BAT60JFILM, Diode_SMD:D_SOD-323_HandSoldering, symbol Device:D_Schottky
- removed D4: BLUELED, Diode_SMD:D_0805_2012Metric_Pad1.15x1.40mm_HandSolder, symbol Device:LED
- removed F1: 500mA, Fuse:Fuse_0603_1608Metric_Pad1.05x0.95mm_HandSolder, symbol Device:Fuse
- removed FB1: 120R, Inductor_SMD:L_0603_1608Metric_Pad1.05x0.95mm_HandSolder, symbol Device:FerriteBead
- removed J1: USB_C_Receptacle_USB2.0_14P, Connector_USB:USB_C_Receptacle_G-Switch_GT-USB-7010ASV, symbol Connector:USB_C_Receptacle_USB2.0_14P
- removed J6: Conn_02x05_Odd_Even, Connector_PinHeader_2.54mm:PinHeader_2x05_P2.54mm_Vertical, symbol Connector_Generic:Conn_02x05_Odd_Even
- removed J7, J8: Conn_01x02_Pin, Connector_PinSocket_2.54mm:PinSocket_1x02_P2.54mm_Vertical, symbol Connector:Conn_01x02_Pin
- removed R1, R10, R4, R5, R9: 150Ω, Resistor_SMD:R_0603_1608Metric_Pad0.98x0.95mm_HandSolder, symbol Device:R_US
- removed R2, R3: 10k, Resistor_SMD:R_0603_1608Metric_Pad0.98x0.95mm_HandSolder, symbol Device:R_US
- removed R6, R7, R8: 10kΩ, Resistor_SMD:R_0603_1608Metric_Pad0.98x0.95mm_HandSolder, symbol Device:R_US
- removed SW1, SW2: SW_SPST, Button_Switch_SMD:SW_SPST_SKQG_WithoutStem, symbol Switch:SW_SPST
- removed U1: FT232RL, Package_SO:SSOP-28_5.3x10.2mm_P0.65mm, symbol Interface_USB:FT232RL
- removed U3: STM32F091RCTx, Package_QFP:LQFP-64_10x10mm_P0.5mm, symbol MCU_ST_STM32F0:STM32F091RCTx
- added J11, J12: Conn_01x30_Pin, symbol Connector:Conn_01x30_Pin
- added J13: Conn_01x06_Socket, symbol Connector:Conn_01x06_Socket
- added JP1: SolderJumper_3_Open, Jumper:SolderJumper-3_P1.3mm_Open_Pad1.0x1.5mm, symbol Jumper:SolderJumper_3_Open
Connections:
- net +3.3V: now also J11.10 (Pin_10), J12.21 (Pin_21)
- net +5V: now also U6.4 (EN), J11.30 (Pin_30), J12.1 (Pin_1), JP1.2 (C); no longer F4.1
- net BRUZ_NCS_0: now also J11.5 (Pin_5)
- net BRUZ_NCS_1: now also J11.4 (Pin_4)
- net BRUZ_NRST: now also J12.10 (Pin_10)
- net GND: now also J11.1 (Pin_1), J12.3 (Pin_3), J12.30 (Pin_30), J13.6 (Pin_6)
- net MT_AX0: now also J12.25 (Pin_25)
- net MT_AX1: now also J12.24 (Pin_24)
- net MT_AX2: now also J12.23 (Pin_23)
- net MT_AX3: now also J12.22 (Pin_22)
- net MT_AY0: now also J12.28 (Pin_28)
- net MT_AY1: now also J12.27 (Pin_27)
- net MT_AY2: now also J12.26 (Pin_26)
- net MT_CS_0: now also J11.7 (Pin_7)
- net MT_CS_1: now also J11.6 (Pin_6)
- net MT_DAT: now also J12.29 (Pin_29)
- net MT_RST: now also J11.3 (Pin_3)
- net MT_STB: now also J11.2 (Pin_2)
- net PC2: now also J11.24 (Pin_24)
- net PC3: now also J11.23 (Pin_23)
- net SPI1_MOSI renamed PA7
- net PA7: now also J12.13 (Pin_13)
- net SPI1_SCK renamed PA5
- net PA5: now also J12.15 (Pin_15)
- new net CTS: J13.5 (Pin_5)
- new net DTR: J13.1 (Pin_1)
- new net NRST_Micro: J12.2 (Pin_2)
- new net PA0: J12.20 (Pin_20)
- new net PA1: J12.19 (Pin_19)
- new net PA11: J12.9 (Pin_9)
- new net PA12: J12.8 (Pin_8)
- new net PA13: J12.7 (Pin_7)
- new net PA14: J12.6 (Pin_6)
- new net PA15: J12.5 (Pin_5)
- new net PA2: J12.18 (Pin_18)
- new net PA3: J12.17 (Pin_17)
- new net PA4: J12.16 (Pin_16)
- new net PA6: J12.14 (Pin_14)
- new net PA8: J12.12 (Pin_12)
- new net PA9: J12.11 (Pin_11)
- new net PB0: J11.9 (Pin_9)
- new net PB1: J11.8 (Pin_8)
- new net PC0: J11.26 (Pin_26)
- new net PC1: J11.25 (Pin_25)
- new net PC10: J11.16 (Pin_16)
- new net PC11: J11.15 (Pin_15)
- new net PC12: J11.14 (Pin_14), J13.2 (Pin_2)
- new net PC13: J11.13 (Pin_13)
- new net PC14: J11.12 (Pin_12)
- new net PC15: J11.11 (Pin_11)
- new net PC4: J11.22 (Pin_22)
- new net PC5: J11.21 (Pin_21)
- new net PC6: J11.20 (Pin_20)
- new net PC7: J11.19 (Pin_19)
- new net PC8: J11.18 (Pin_18)
- new net PC9: J11.17 (Pin_17)
- new net PD2: J12.4 (Pin_4), J13.3 (Pin_3)
- new net PF0: J11.29 (Pin_29)
- new net PF1: J11.28 (Pin_28)
- new net PF11: J11.27 (Pin_27)
- new net POWER_5V: F4.1, JP1.1 (A)
- new net USB_5V: J13.4 (Pin_4), JP1.3 (B)
- no-connect marks 47 -> 9
Other:
- note added: "MicroController PinOuts"
- note added: "Wall Adaptor and Power Jumper"
- note removed: "Micro Status LEDs"
- note removed: "UART Status LEDs"
- note removed: "Wall Adaptor"
- moved on the sheet: C13, J9

Commit message: Parker Loves Furries
Parts:
- removed U4, U5: CD22M3494MQZ, SeniorDesign:PLCC44_16P66X16P66_INR-M, symbol SeniorDesign:CD22M3494MQZ
- added U1, U2: DIP, Package_DIP:DIP-40_W15.24mm, symbol SeniorDesign:MTT8816DIP
- C12: renamed from C23; footprint Capacitor_SMD:C_0201_0603Metric_Pad0.64x0.40mm_HandSolder -> Capacitor_SMD:C_0603_1608Metric
- C15: renamed from C26; footprint Capacitor_SMD:C_0201_0603Metric_Pad0.64x0.40mm_HandSolder -> Capacitor_SMD:C_0805_2012Metric
- C9: renamed from C20; footprint Capacitor_SMD:C_0201_0603Metric_Pad0.64x0.40mm_HandSolder -> Capacitor_SMD:C_0603_1608Metric
- J5: renamed from J11; footprint (none) -> Connector_PinSocket_2.54mm:PinSocket_1x30_P2.54mm_Vertical
- J6: renamed from J12; footprint (none) -> Connector_PinSocket_2.54mm:PinSocket_1x30_P2.54mm_Vertical
- J7: renamed from J13; footprint (none) -> Connector_PinSocket_2.54mm:PinSocket_1x06_P2.54mm_Vertical
- U4: renamed from U8; footprint SeniorDesign:SOP65P640X120-24N -> Package_DIP:DIP-24_W15.24mm
- U6: renamed from U7; footprint SeniorDesign:SOP65P640X120-24N -> Package_DIP:DIP-24_W15.24mm
- renumbered C12 to C1, C21 to C10, C22 to C11, C24 to C13, C25 to C14, C27 to C16, C28 to C17, C29 to C18, C13 to C2, C14 to C3, C15 to C4, C16 to C5, C17 to C6, C18 to C7, C19 to C8, F2 to F1, F3 to F2, F4 to F3, J2 to J1, J3 to J2, J4 to J3, J5 to J4, J9 to J8, R11 to R1, R12 to R2, R13 to R3, R14 to R4, R15 to R5, R16 to R6, R17 to R7, U2 to U3, U6 to U5, U9 to U7, U10 to U8
Connections:
- net +5V: now also U1.40 (VDD), U2.40 (VDD)
- net -5V: now also U1.20 (VEE), U2.20 (VEE)
- net GND: now also U1.16 (VSS), U2.16 (VSS)
- net MT_AX0: now also U1.5 (AX0), U2.5 (AX0)
- net MT_AX1: now also U1.22 (AX1), U2.22 (AX1)
- net MT_AX2: now also U1.23 (AX2), U2.23 (AX2)
- net MT_AX3: now also U1.4 (AX3), U2.4 (AX3)
- net MT_AY0: now also U1.24 (AY0), U2.24 (AY0)
- net MT_AY1: now also U1.25 (AY1), U2.25 (AY1)
- net MT_AY2: now also U1.2 (AY2), U2.2 (AY2)
- net MT_CS_0: now also U2.36 (CS)
- net MT_CS_1: now also U1.36 (CS)
- net MT_DAT: now also U1.38 (DATA), U2.38 (DATA)
- net MT_RST: now also U1.3 (RESET), U2.3 (RESET)
- net MT_STB: now also U1.18 (STROBE), U2.18 (STROBE)
- net CTS: no longer names the net of J7.5 (Pin_5)
- net DTR: no longer names the net of J7.1 (Pin_1)
- net NRST_Micro: no longer names the net of J6.2 (Pin_2)
- net PA0: no longer names the net of J6.20 (Pin_20)
- net PA1: no longer names the net of J6.19 (Pin_19)
- net PA11: no longer names the net of J6.9 (Pin_9)
- net PA12: no longer names the net of J6.8 (Pin_8)
- net PA13: no longer names the net of J6.7 (Pin_7)
- net PA14: no longer names the net of J6.6 (Pin_6)
- net PA15: no longer names the net of J6.5 (Pin_5)
- net PA2: no longer names the net of J6.18 (Pin_18)
- net PA3: no longer names the net of J6.17 (Pin_17)
- net PA4: no longer names the net of J6.16 (Pin_16)
- net PA6: no longer names the net of J6.14 (Pin_14)
- net PA8: no longer names the net of J6.12 (Pin_12)
- net PA9: no longer names the net of J6.11 (Pin_11)
- net PB0: no longer names the net of J5.9 (Pin_9)
- net PB1: no longer names the net of J5.8 (Pin_8)
- net PC0: no longer names the net of J5.26 (Pin_26)
- net PC1: no longer names the net of J5.25 (Pin_25)
- net PC10: no longer names the net of J5.16 (Pin_16)
- net PC11: no longer names the net of J5.15 (Pin_15)
- net PC13: no longer names the net of J5.13 (Pin_13)
- net PC14: no longer names the net of J5.12 (Pin_12)
- net PC15: no longer names the net of J5.11 (Pin_11)
- net PC2: no longer names the net of J5.24 (Pin_24)
- net PC3: no longer names the net of J5.23 (Pin_23)
- net PC4: no longer names the net of J5.22 (Pin_22)
- net PC5: no longer names the net of J5.21 (Pin_21)
- net PC6: no longer names the net of J5.20 (Pin_20)
- net PC7: no longer names the net of J5.19 (Pin_19)
- net PC8: no longer names the net of J5.18 (Pin_18)
- net PC9: no longer names the net of J5.17 (Pin_17)
- net PF0: no longer names the net of J5.29 (Pin_29)
- net PF1: no longer names the net of J5.28 (Pin_28)
- net PF11: no longer names the net of J5.27 (Pin_27)
- no-connect marks 9 -> 45
Other:
- moved on the sheet: U4A, U6A

Commit message: I know of at least one
Parts:
- removed C10: 15n, Capacitor_SMD:C_0402_1005Metric_Pad0.74x0.62mm_HandSolder, symbol Device:C
- removed C13, C14: 100nF, Capacitor_SMD:C_0402_1005Metric_Pad0.74x0.62mm_HandSolder, symbol Device:C
- removed C15: 1µF, Capacitor_SMD:C_0805_2012Metric, symbol Device:C
- removed C17: 10µF, Capacitor_SMD:C_1210_3225Metric_Pad1.33x2.70mm_HandSolder, symbol Device:C
- removed C18: 33u, Capacitor_Tantalum_SMD:CP_EIA-3528-21_Kemet-B_HandSolder, symbol Device:C
- removed C4: 22u, SeniorDesign:CAP_EEFK_C_PAN, symbol Device:C_Polarized
- removed C5: 4.7u, Capacitor_SMD:C_1210_3225Metric_Pad1.33x2.70mm_HandSolder, symbol Device:C
- removed C6: 1µF, Capacitor_SMD:C_0402_1005Metric_Pad0.74x0.62mm_HandSolder, symbol Device:C
- removed C8: 240p, Capacitor_SMD:C_0402_1005Metric_Pad0.74x0.62mm_HandSolder, symbol Device:C
- removed C9: 4.7u, Capacitor_SMD:C_0603_1608Metric, symbol Device:C
- removed L2: 10u, Inductor_SMD:L_Bourns_SRN6045TA, symbol Device:L
- removed R1: 24.9k, Resistor_SMD:R_0402_1005Metric_Pad0.72x0.64mm_HandSolder, symbol Device:R_US
- removed R2: 261k, Resistor_SMD:R_0402_1005Metric_Pad0.72x0.64mm_HandSolder, symbol Device:R_US
- removed R3: 100k, Resistor_SMD:R_0402_1005Metric_Pad0.72x0.64mm_HandSolder, symbol Device:R_US
- removed R4: 8.87k, Resistor_SMD:R_0402_1005Metric_Pad0.72x0.64mm_HandSolder, symbol Device:R_US
- removed R7: 6.04k, Resistor_SMD:R_0402_1005Metric_Pad0.72x0.64mm_HandSolder, symbol Device:R_US
- removed Rfbt1: 102k, Resistor_SMD:R_0402_1005Metric_Pad0.72x0.64mm_HandSolder, symbol Device:R_US
- removed U7: XTPS55285VALR, SeniorDesign:TPS55285, symbol SeniorDesign:XTPS55285VALR
- C7: footprint Capacitor_SMD:C_1210_3225Metric_Pad1.33x2.70mm_HandSolder -> Capacitor_SMD:C_0805_2012Metric_Pad1.18x1.45mm_HandSolder
- JP1: footprint Jumper:SolderJumper-3_P1.3mm_Open_Pad1.0x1.5mm -> Jumper:SolderJumper-3_P1.3mm_Open_Pad1.0x1.5mm_NumberLabels
- U5, U8: footprint Package_TO_SOT_SMD:SOT-23-6 -> Connector_PinHeader_2.54mm:PinHeader_1x06_P2.54mm_Vertical
Connections:
- net +5V: now also C7.2, F3.2, U8.3 (VIN); no longer JP1.2 (C)
- net BRUZ_NCS_0: now also J6.18 (Pin_18); no longer J5.5 (Pin_5)
- net BRUZ_NCS_1: now also J6.16 (Pin_16); no longer J5.4 (Pin_4)
- net BRUZ_NRST: now also J6.17 (Pin_17)
- net MT_AX0: now also J6.23 (Pin_23); no longer J6.25 (Pin_25)
- net MT_AX1: now also J5.2 (Pin_2); no longer J6.24 (Pin_24)
- net MT_AX2: now also J5.3 (Pin_3); no longer J6.23 (Pin_23)
- net MT_AX3: now also J6.24 (Pin_24); no longer J6.22 (Pin_22)
- net MT_AY0: now also J5.6 (Pin_6); no longer J6.28 (Pin_28)
- net MT_AY1: now also J6.29 (Pin_29); no longer J6.27 (Pin_27)
- net MT_CS_0: now also J6.19 (Pin_19); no longer J5.7 (Pin_7)
- net MT_CS_1: now also J6.28 (Pin_28); no longer J5.6 (Pin_6)
- net MT_DAT: now also J6.20 (Pin_20), J6.27 (Pin_27); no longer J6.29 (Pin_29)
- net MT_RST: now also J6.25 (Pin_25); no longer J5.3 (Pin_3)
- net MT_STB: now also J6.22 (Pin_22); no longer J5.2 (Pin_2)
- net WallAdpt: now also JP1.1 (A); no longer C7.2, U8.3 (VIN)
- net POWER_5V: no longer names the net of F3.1
- net POWER_5V: now also JP1.2 (C); no longer JP1.1 (A)
- new net PB4: J5.5 (Pin_5)
- new net PB5: J5.4 (Pin_4)
- no-connect marks 45 -> 39
Other:
- note removed: "Switching Buck-Boost Converter"
- moved on the sheet: F3

Commit message: PCB done
Parts:
- U1, U2: footprint Package_DIP:DIP-40_W15.24mm -> Package_DIP:DIP-40_W15.24mm_LongPads
Changed lines of the file:
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@@
 			)
 		)
-		(property "Footprint" "Package_DIP:DIP-40_W15.24mm"
+		(property "Footprint" "Package_DIP:DIP-40_W15.24mm_LongPads"
 			(at 72.39 156.21 0)
 			(effects
@@
 			)
 		)
-		(property "Footprint" "Package_DIP:DIP-40_W15.24mm"
+		(property "Footprint" "Package_DIP:DIP-40_W15.24mm_LongPads"
 			(at 74.93 238.76 0)
 			(effects
@@
 					(size 1.27 1.27)
 				)
-				(hide yes)
 			)
 		)
