File: hardware/SignleCellBoard/untitled.kicad_sch (KiCad schematic)
At the start: 13 parts, among them J10 Conn_01x02_Pin, U11 TL071, U12 TL071, U4 CD22M3494MQZ, U5 CD22M3494MQZ, U7 AD5263BRUZ200, U8 AD5263BRUZ200

Commit message: Parker Loves Furries
Parts:
- removed U4, U5: CD22M3494MQZ, SeniorDesign:PLCC44_16P66X16P66_INR-M, symbol SeniorDesign:CD22M3494MQZ
- added U1, U2: DIP, Package_DIP:DIP-40_W15.24mm, symbol SeniorDesign:MTT8816DIP
- U4: renamed from U8; footprint SeniorDesign:SOP65P640X120-24N -> Package_DIP:DIP-24_W15.24mm; DKPN AD5263BRUZ200-R7 -> (none); MPN (none) -> AD5263BRUZ200
- U6: renamed from U7; footprint SeniorDesign:SOP65P640X120-24N -> Package_DIP:DIP-24_W15.24mm
- renumbered C30 to C19, C31 to C20, C32 to C21, C33 to C22, D7 to D1, D8 to D2, J10 to J9, U12 to U10, U11 to U9
Connections:
- net C1_in: now also U2.10 (X8)
- net C1_out: now also U2.11 (X9)
- net C2_in: now also U1.6 (X14)
- net C2_out: now also U1.7 (X15)
- net C3_in: now also U2.7 (X15)
- net C3_out: now also U2.6 (X14)
- net C4_in: now also U2.13 (X11)
- net C4_out: now also U2.12 (X10)
- net D1_anode: now also U2.9 (X7)
- net D1_cathode: now also U2.8 (X6)
- net D2_anode: now also U1.26 (X13)
- net D2_cathode: now also U1.27 (X12)
- net GND: now also U1.21 (Y4), U2.35 (Y0)
- net Input_1: now also U1.35 (Y0), U2.15 (Y7)
- net Input_2: now also U1.37 (Y1), U2.17 (Y6)
- net Input_3: now also U1.39 (Y2), U2.19 (Y5)
- net J1_in: now also U1.8 (X6)
- net J1_out: now also U1.9 (X7)
- net Op1_neg: now also U1.30 (X3)
- net Op1_out: now also U1.28 (X5)
- net Op1_pos: now also U1.29 (X4)
- net Op2_neg: now also U1.33 (X0)
- net Op2_out: now also U1.31 (X2)
- net Op2_pos: now also U1.32 (X1)
- net Output: now also U1.1 (Y3), U2.1 (Y3)
- net R1_in: now also U2.30 (X3)
- net R1_out: now also U2.31 (X2)
- net R2_in: now also U1.10 (X8)
- net R2_out: now also U1.11 (X9)
- net R3_in: now also U2.32 (X1)
- net R3_out: now also U2.33 (X0)
- net R4_in: now also U1.12 (X10)
- net R4_out: now also U1.13 (X11)
- net R5_in: now also U2.26 (X13)
- net R5_out: now also U2.27 (X12)
- net R6_in: now also U2.28 (X5)
- net R6_out: now also U2.29 (X4)
- net Y5: now also U1.19 (Y5), U2.37 (Y1)
- net Y6: now also U1.17 (Y6), U2.39 (Y2)
- net Y7: now also U1.15 (Y7), U2.21 (Y4)

Commit message: I know of at least one
Connections:
- net D2_anode: now also U1.9 (X7); no longer U1.26 (X13)
- net D2_cathode: now also U1.8 (X6); no longer U1.27 (X12)
- net J1_in: now also U1.27 (X12); no longer U1.8 (X6)
- net J1_out: now also U1.26 (X13); no longer U1.9 (X7)
- net Op2_neg: now also U1.32 (X1); no longer U1.33 (X0)
- net Op2_out: now also U1.33 (X0); no longer U1.31 (X2)
- net Op2_pos: now also U1.31 (X2); no longer U1.32 (X1)
Changed lines of the file:
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@@
 	)
 	(label "Op2_neg"
-		(at 128.27 107.95 180)
+		(at 128.27 110.49 180)
 		(effects
 			(font
@@
 	)
 	(label "D2_cathode"
-		(at 128.27 138.43 180)
+		(at 128.27 123.19 180)
 		(effects
 			(font
@@
 	)
 	(label "J1_out"
-		(at 128.27 125.73 180)
+		(at 128.27 140.97 180)
 		(effects
 			(font
@@
 	)
 	(label "Op2_pos"
-		(at 128.27 110.49 180)
+		(at 128.27 113.03 180)
 		(effects
 			(font
@@
 	)
 	(label "D2_anode"
-		(at 128.27 140.97 180)
+		(at 128.27 125.73 180)
 		(effects
 			(font
@@
 	)
 	(label "Op2_out"
-		(at 128.27 113.03 180)
+		(at 128.27 107.95 180)
 		(effects
 			(font
@@
 	)
 	(label "J1_in"
-		(at 128.27 123.19 180)
-		(effects
-			(font
+		(at 128.27 138.43 180)
+		(effects
+			(font

Commit message: PCB done
Parts:
- U1, U2: footprint Package_DIP:DIP-40_W15.24mm -> Package_DIP:DIP-40_W15.24mm_LongPads
Changed lines of the file:
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@@
 			)
 		)
-		(property "Footprint" "Package_DIP:DIP-40_W15.24mm"
+		(property "Footprint" "Package_DIP:DIP-40_W15.24mm_LongPads"
 			(at 151.13 121.92 0)
 			(effects
@@
 			)
 		)
-		(property "Footprint" "Package_DIP:DIP-40_W15.24mm"
+		(property "Footprint" "Package_DIP:DIP-40_W15.24mm_LongPads"
 			(at 214.63 123.19 0)
 			(effects
